File: SlaveDesignFiles/sheet1.kicad_pcb (KiCad board)
At the start: 4 copper layers, 216 x 144 mm, 569 parts, among them CN1 DB141V-2.54-6P, CN2 DB141V-2.54-6P, CN3 X3025WVS-2*10D-LPSW, CN4 X3025WVS-2*10D-LPSW, CN5 X3025WVS-2*10D-LPSW, CN6 X3025WVS-2*10D-LPSW, CN7 DB141V-2.54-6P, CN8 DB141V-2.54-6P, J1 Conn_02x02_Counter_Clockwise, J2 Conn_02x02_Counter_Clockwise, J3 2.54-2*5, J4 2.54-2*5, J5 2.54-2*5, J6 2.54-2*5, J7 PM2.54-2*10, J8 2.54-2*5, M1 Conn_01x01_Socket, M2 Conn_01x01_Socket, M3 Conn_01x01_Socket, M4 Conn_01x01_Socket, M5 Conn_01x01_Socket, M6 Conn_01x01_Socket, M7 Conn_01x01_Socket, M8 Conn_01x01_Socket, Q1 TXB0104PWR, Q10 TPT75176B-SO1R, Q11 SDT23C712L02_C5197393, Q12 SDT23C712L02_C5197393, Q13 TXB0104PWR, Q14 TPS27082LDDCR, Q15 TPT75176B-SO1R, Q16 TPT75176B-SO1R, Q17 SDT23C712L02_C5197393, Q18 SDT23C712L02_C5197393, Q19 TXB0104PWR, Q2 TPS27082LDDCR, Q20 TPS27082LDDCR, Q21 TPT75176B-SO1R, Q22 TPT75176B-SO1R, Q23 SDT23C712L02_C5197393, Q24 SDT23C712L02_C5197393, Q25 DP83822IRHBR, Q26 DP83822IRHBR, Q27 SDT23C712L02_C5197393, Q28 SDT23C712L02_C5197393, Q29 SDT23C712L02_C5197393, Q3 TPT75176B-SO1R, Q30 AM26C32CD, Q31 SDT23C712L02_C5197393, Q32 SDT23C712L02_C5197393, Q33 SDT23C712L02_C5197393, Q34 AM26C32CD, Q35 TPT75176B-SO1R, Q36 SN74LVC1G125DCKR, Q37 SDT23C712L02_C5197393, Q38 AMCW3225P-2-242T, Q39 TPT75176B-SO1R, Q4 TPT75176B-SO1R, Q40 SN74LVC1G125DCKR, Q41 SDT23C712L02_C5197393, Q42 AMCW3225P-2-242T, Q43 SN74ACT244PWRG4, Q44 SN74ACT244PWRG4, Q45 SN74ACT244PWRG4, Q46 SN74ACT244PWRG4, Q47 FMMT618TA, Q48 FMMT618TA, Q49 FMMT618TA, Q5 SDT23C712L02_C5197393, Q50 SN74LVC14APWRG4, Q51 FMMT618TA, Q52 TPT1042VQ-SO1R-S, Q53 TPT1042VQ-SO1R-S, Q54 SDT23C712L02_C5197393, Q55 SDT23C712L02_C5197393, Q56 CP2102N-A02-GQFN28R, Q57 TYPEC-304-ACP16, Q58 AT24C16C-SSHM-T, Q59 SRV05-4HTG, Q6 SDT23C712L02_C5197393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

Commit message: First version
Parts:
- removed the D2 at (209.6, 151.6)
- removed the D4 at (216.4, 173.6)
- removed the D6 at (98.9, 151.5)
- removed the D8 at (99.5, 184.6)
- removed Q57: TYPEC-304-ACP16, Lib4:USB-C-SMD_TYPE-C-16P-1
- removed the R192 at (209.6, 153.5)
- removed the R194 at (222.2, 154.3)
- removed the R208 at (216.5, 180.5)
- removed the R234 at (99.3, 182.6)
- removed the R236 at (87.7, 180.6)
- removed TP1, TP2: TestPoint, TestPoint:TestPoint_Loop_D2.60mm_Drill1.4mm_Beaded
- added C107: 15pF/50V, Capacitor_SMD:C_0603_1608Metric, F.Cu at (220.3, 143.5)
- added C108: 0.01uF/50V, Capacitor_SMD:C_0603_1608Metric, F.Cu at (218.2, 140.2)
- added C110: 15pF/50V, Capacitor_SMD:C_0603_1608Metric, F.Cu at (235.9, 182.1)
- added C111: 0.01uF/50V, Capacitor_SMD:C_0603_1608Metric, F.Cu at (238.0, 185.4)
- added C113: 15pF/50V, Capacitor_SMD:C_0603_1608Metric, F.Cu at (74.8, 142.6)
- added C114: 0.01uF/50V, Capacitor_SMD:C_0603_1608Metric, F.Cu at (72.7, 139.3)
- added C116: 15pF/50V, Capacitor_SMD:C_0603_1608Metric, F.Cu at (69.6, 178.4)
- added C117: 0.01uF/50V, Capacitor_SMD:C_0603_1608Metric, F.Cu at (67.5, 175.1)
- added D18: LEDRED, LED_SMD:LED_0805_2012Metric, F.Cu at (234.3, 140.2)
- added D20: LEDRED, LED_SMD:LED_0805_2012Metric, F.Cu at (234.6, 188.5)
- added D22: LEDRED, LED_SMD:LED_0805_2012Metric, F.Cu at (80.2, 136.3)
- added D24: LEDRED, LED_SMD:LED_0805_2012Metric, F.Cu at (78.8, 170.0)
- added D37: SK36A-LTP, Lib_sheet_10:SMA_L4.3-W2.6-LS5.2-RD, F.Cu at (171.6, 226.3)
- added Q25: SN74LVC1G125DCKR, Lib2ic:SOT-353_L2.2-W1.4-P0.65-LS2.4-BR, F.Cu at (220.3, 140.2)
- added Q27: FMMT618TA, Package_TO_SOT_SMD:SOT-23, F.Cu at (229.1, 140.2)
- added Q28: SN74LVC1G125DCKR, Lib2ic:SOT-353_L2.2-W1.4-P0.65-LS2.4-BR, F.Cu at (235.9, 185.4)
- added Q30: FMMT618TA, Package_TO_SOT_SMD:SOT-23, F.Cu at (227.1, 185.4)
- added Q31: SN74LVC1G125DCKR, Lib2ic:SOT-353_L2.2-W1.4-P0.65-LS2.4-BR, F.Cu at (74.8, 139.3)
- added Q33: FMMT618TA, Package_TO_SOT_SMD:SOT-23, F.Cu at (83.6, 139.3)
- added Q34: SN74LVC1G125DCKR, Lib2ic:SOT-353_L2.2-W1.4-P0.65-LS2.4-BR, F.Cu at (69.6, 175.1)
- added Q36: FMMT618TA, Package_TO_SOT_SMD:SOT-23, F.Cu at (78.4, 175.1)
- added Q46: TYPEC-304-ACP16, Lib4:USB-C-SMD_TYPE-C-16P-1, F.Cu at (180.9, 234.0)
- added R187: 3.3K, Lib_sheet_10:R_0603_1608Metric, F.Cu at (223.2, 144.3)
- added R188: 470R, Resistor_SMD:R_0603_1608Metric, F.Cu at (223.2, 142.7)
- added R195: 62R/1%, Resistor_SMD:R_0603_1608Metric, F.Cu at (222.3, 140.2)
- added R202: 10K, Resistor_SMD:R_0805_2012Metric, F.Cu at (224.1, 140.2)
- added R203: 2K, Resistor_SMD:R_0805_2012Metric, F.Cu at (226.1, 140.2)
- added R204: 1K, Resistor_SMD:R_0805_2012Metric, F.Cu at (232.2, 140.2)
- added R205: 3.3K, Lib_sheet_10:R_0603_1608Metric, F.Cu at (233.0, 181.3)
- added R213: 62R/1%, Resistor_SMD:R_0603_1608Metric, F.Cu at (233.9, 185.4)
- added R221: 2K, Resistor_SMD:R_0805_2012Metric, F.Cu at (230.1, 185.4)
- added R223: 3.3K, Lib_sheet_10:R_0603_1608Metric, F.Cu at (77.7, 143.4)
- added R224: 470R, Resistor_SMD:R_0603_1608Metric, F.Cu at (77.7, 141.8)
- added R231: 62R/1%, Resistor_SMD:R_0603_1608Metric, F.Cu at (76.8, 139.3)
- added R238: 10K, Resistor_SMD:R_0805_2012Metric, F.Cu at (78.6, 139.3)
- added R239: 2K, Resistor_SMD:R_0805_2012Metric, F.Cu at (80.6, 139.3)
- added R240: 1K, Resistor_SMD:R_0805_2012Metric, F.Cu at (83.7, 136.4)
- added R241: 3.3K, Lib_sheet_10:R_0603_1608Metric, F.Cu at (72.5, 179.2)
- added R242: 470R, Resistor_SMD:R_0603_1608Metric, F.Cu at (72.5, 177.7)
- added R249: 62R/1%, Resistor_SMD:R_0603_1608Metric, F.Cu at (71.6, 175.1)
- added R256: 10K, Resistor_SMD:R_0805_2012Metric, F.Cu at (73.4, 175.1)
- added R257: 2K, Resistor_SMD:R_0805_2012Metric, F.Cu at (75.4, 175.1)
- added R258: 1K, Resistor_SMD:R_0805_2012Metric, F.Cu at (78.7, 172.2)
- added ref1: Conn_01x01_Socket, 1mmlab_footprint:Mark_TH_3mm, F.Cu at (54.7, 241.2)
- added ref10: Conn_01x01_Socket, 1mmlab_footprint:Mark_SMD, B.Cu at (244.7, 241.2)
- added ref11: Conn_01x01_Socket, 1mmlab_footprint:Mark_SMD, F.Cu at (59.7, 93.2)
- added ref12: Conn_01x01_Socket, 1mmlab_footprint:Mark_SMD, F.Cu at (244.7, 93.2)
- added ref13: Conn_01x01_Socket, 1mmlab_footprint:Mark_SMD, B.Cu at (82.0, 110.8)
- added ref14: Conn_01x01_Socket, 1mmlab_footprint:Mark_SMD, B.Cu at (72.3, 222.1)
- added ref15: Conn_01x01_Socket, 1mmlab_footprint:Mark_SMD, F.Cu at (82.0, 110.8)
- added ref16: Conn_01x01_Socket, 1mmlab_footprint:Mark_SMD, F.Cu at (72.3, 222.1)
- added ref17: Conn_01x01_Socket, 1mmlab_footprint:Mark_SMD, F.Cu at (208.9, 138.3)
- added ref18: Conn_01x01_Socket, 1mmlab_footprint:Mark_SMD, F.Cu at (242.3, 219.4)
- added ref19: Conn_01x01_Socket, 1mmlab_footprint:Mark_SMD, B.Cu at (242.3, 219.4)
- added ref2: Conn_01x01_Socket, 1mmlab_footprint:Mark_TH_3mm, F.Cu at (254.7, 241.2)
- added ref20: Conn_01x01_Socket, 1mmlab_footprint:Mark_SMD, B.Cu at (208.9, 138.3)
- added ref3: Conn_01x01_Socket, 1mmlab_footprint:Mark_TH_3mm, F.Cu at (54.7, 93.2)
- added ref4: Conn_01x01_Socket, 1mmlab_footprint:Mark_TH_3mm, F.Cu at (254.7, 93.2)
- added ref5: Conn_01x01_Socket, 1mmlab_footprint:Mark_SMD, B.Cu at (244.7, 93.2)
- added ref6: Conn_01x01_Socket, 1mmlab_footprint:Mark_SMD, B.Cu at (59.7, 93.2)
- added ref7: Conn_01x01_Socket, 1mmlab_footprint:Mark_SMD, F.Cu at (59.7, 241.2)
- added ref8: Conn_01x01_Socket, 1mmlab_footprint:Mark_SMD, F.Cu at (244.7, 241.2)
- added ref9: Conn_01x01_Socket, 1mmlab_footprint:Mark_SMD, B.Cu at (59.7, 241.2)
- C134: renamed from C126; moved to B.Cu
- C135: renamed from C127; moved to B.Cu
- R206: value 20K/1% -> 470R
- R220: value 20K/1% -> 10K; footprint Resistor_SMD:R_0603_1608Metric -> Resistor_SMD:R_0805_2012Metric
- R222: value 20K/1% -> 1K; footprint Resistor_SMD:R_0603_1608Metric -> Resistor_SMD:R_0805_2012Metric
- X1, X2: moved to B.Cu
- moved Q45 200.1 mm to (231.1, 226.1), turned to 180 degrees
- moved C138 189.8 mm to (238.0, 224.6), turned to 90 degrees
- moved C140 187.3 mm to (236.5, 224.6), turned to -90 degrees
- moved C143 181.2 mm to (223.0, 226.9)
- moved C142 181.2 mm to (224.6, 226.9)
- moved C144 179.5 mm to (217.5, 226.9)
- moved R220 154.3 mm to (232.1, 185.4), turned to 90 degrees
- moved R222 142.6 mm to (231.1, 188.5)
- moved Q42 106.2 mm to (82.6, 192.3), turned to 90 degrees
- moved C135 65.5 mm to (141.0, 192.1)
- moved X2 59.4 mm to (144.1, 192.2), turned to 0 degrees
- moved D31 32.4 mm to (86.5, 220.9)
- moved C126 30.3 mm to (87.2, 192.3), turned to -90 degrees
- moved C127 26.6 mm to (87.2, 165.7)
- moved C134 26.0 mm to (227.6, 190.2)
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- renumbered C107 to C109, C108 to C112, C109 to C115, C110 to C118, C111 to C119, C112 to C120, C113 to C121, C114 to C122, C115 to C123, C116 to C124, C117 to C125, C118 to C126, C119 to C127, C120 to C128, C121 to C129, C122 to C130, C123 to C131, C124 to C132, C125 to C133, C128 to C136, C129 to C137, C130 to C138, C131 to C139, C132 to C140, C133 to C141, C134 to C142, C135 to C143, C136 to C144, C137 to C145, Q5 to D1, Q28 to D10, Q29 to D11, Q31 to D12, Q32 to D13, Q33 to D14, Q37 to D15, Q41 to D16, D1 to D17, D3 to D19, Q6 to D2, D5 to D21, D7 to D23, D9 to D25, D10 to D26, D11 to D27, D12 to D28, D13 to D29, Q11 to D3, D14 to D30, D15 to D31, Q54 to D32, Q55 to D33, D16 to D34, D17 to D35, D18 to D36, D19 to D38, D20 to D39, Q12 to D4, D21 to D40, D22 to D41, Q17 to D5, Q18 to D6, Q23 to D7, Q24 to D8, Q27 to D9, Q38 to L15, Q42 to L16, L15 to L17, L16 to L18, L17 to L19, Q14 to Q10, Q15 to Q11, Q16 to Q12, Q19 to Q13, Q20 to Q14, Q21 to Q15, Q22 to Q16, Q25 to Q17, Q26 to Q18, Q30 to Q19, Q34 to Q20, Q35 to Q21, Q36 to Q22, Q39 to Q23, Q40 to Q24, Q43 to Q26, Q44 to Q29, Q45 to Q32, Q46 to Q35, Q47 to Q37, Q48 to Q38, Q49 to Q39, Q50 to Q40, Q51 to Q41, Q52 to Q42, Q53 to Q43, Q56 to Q44, U8 to Q45, Q58 to Q47, Q59 to Q48, Q7 to Q5, Q8 to Q6, Q9 to Q7, Q10 to Q8, Q13 to Q9, R187 to R189, R188 to R190, R189 to R191, R190 to R192, R191 to R193, R193 to R194, R195 to R196, R196 to R197, R197 to R198, R198 to R199, R199 to R200, R200 to R201, R201 to R207, R202 to R208, R203 to R209, R204 to R210, R205 to R211, R207 to R212, R209 to R214, R210 to R215, R211 to R216, R212 to R217, R213 to R218, R214 to R219, R215 to R225, R216 to R226, R217 to R227, R218 to R228, R219 to R229, R221 to R230, R223 to R232, R224 to R233, R225 to R234, R226 to R235, R227 to R236, R228 to R237, R229 to R243, R230 to R244, R231 to R245, R232 to R246, R233 to R247, R235 to R248, R237 to R250, R238 to R251, R239 to R252, R240 to R253, R241 to R254, R242 to R255, R243 to R259, R244 to R260, R245 to R261, R246 to R262, R247 to R263, R248 to R264, R249 to R265, R250 to R266, R251 to R267, R252 to R268, R253 to R269, R254 to R270, R255 to R271, R256 to R272, R257 to R273, R258 to R274, R259 to R275, R260 to R276, R261 to R277, R262 to R278, R263 to R279, R264 to R280, R265 to R281, R266 to R282, R267 to R283, R268 to R284, R269 to R285, R270 to R286, R271 to R287, R272 to R288, R273 to R289, R274 to R290, R275 to R291, R276 to R292, R277 to R293, R278 to R294, R279 to R295, R280 to R296, R281 to R297, R282 to R298, R283 to R299, R284 to R300, R285 to R301, R286 to R302, R287 to R303, R288 to R304, R289 to R305, R290 to R306, R291 to R307, R292 to R308
Connections:
- net /ADC_CLK_1 renamed /ADC_CLK_X1
- net /ADC_CLK_2 renamed /ADC_CLK_X2
- C103 pad 1: D+5V_ -> D+5V
- C109 pad 1: D+5V_ -> D+5V
- C112 pad 1: D+5V_ -> D+5V
- C115 pad 1: D+5V_ -> D+5V
- C118 pad 1: D+5V_ -> D+5V
- C126 pad 1: D+5V_ -> D+5V
- C127 pad 1: D+5V_ -> D+5V
- C138 pad 2: D+5V_ -> D+5V
- C14 pad 1: D+5V_ -> D+5V
- C140 pad 1: D+5V_ -> D+5V
- C142 pad 1: +3.3V -> VDD
- C143 pad 2: +3.3V -> VDD
- C144 pad 1: +3.3V -> VDD
- C15 pad 1: D+5V_ -> D+5V
- C17 pad 2: D+5V_ -> D+5V
- C19 pad 2: D+5V_ -> D+5V
- C2 pad 1: D+5V_ -> D+5V
- C20 pad 2: D+5V_ -> D+5V
- C26 pad 1: D+5V_ -> D+5V
- C27 pad 1: D+5V_ -> D+5V
- C29 pad 2: D+5V_ -> D+5V
- C3 pad 1: D+5V_ -> D+5V
- C31 pad 2: D+5V_ -> D+5V
- C32 pad 2: D+5V_ -> D+5V
- C38 pad 1: D+5V_ -> D+5V
- C39 pad 1: D+5V_ -> D+5V
- C41 pad 2: D+5V_ -> D+5V
- C43 pad 2: D+5V_ -> D+5V
- C44 pad 2: D+5V_ -> D+5V
- C5 pad 2: D+5V_ -> D+5V
- C7 pad 2: D+5V_ -> D+5V
- C8 pad 2: D+5V_ -> D+5V
- C82 pad 1: D+5V_ -> D+5V
- C92 pad 1: D+5V_ -> D+5V
- C96 pad 1: D+5V_ -> D+5V
- CN3 pad 1: D+5V_ -> D+5V
- CN3 pad 15: /IPM_VDC_BUS2 -> /DSP_VDC_BUS2
- CN3 pad 16: /IPM_Temperature2 -> /DSP_Temperature2
- CN3 pad 17: AGND -> /DSP_PWM2_~{FAULT}
- CN3 pad 2: D+5V_ -> D+5V
- CN3 pad 21: unconnected-(CN3-Pad21) -> AGND
- CN3 pad 22: PE_GND -> AGND
- CN4 pad 1: D+5V_ -> D+5V
- CN4 pad 15: /IPM_VDC_BUS1 -> /DSP_VDC_BUS1
- CN4 pad 16: /IPM_Temperature1 -> /DSP_Temperature1
- CN4 pad 17: AGND -> /DSP_PWM1_~{FAULT}
- CN4 pad 2: D+5V_ -> D+5V
- CN4 pad 21: unconnected-(CN4-Pad21) -> AGND
- CN4 pad 22: PE_GND -> AGND
- CN5 pad 1: D+5V_ -> D+5V
- CN5 pad 15: /IPM_VDC_BUS3 -> /DSP_VDC_BUS3
- CN5 pad 16: /IPM_Temperature3 -> /DSP_Temperature3
- CN5 pad 17: AGND -> /DSP_PWM3_~{FAULT}
- CN5 pad 2: D+5V_ -> D+5V
- CN5 pad 21: unconnected-(CN5-Pad21) -> AGND
- CN5 pad 22: PE_GND -> AGND
- CN6 pad 1: D+5V_ -> D+5V
- CN6 pad 15: /IPM_VDC_BUS4 -> /DSP_VDC_BUS4
- CN6 pad 16: /IPM_Temperature4 -> /DSP_Temperature4
- CN6 pad 17: AGND -> /DSP_PWM4_~{FAULT}
- CN6 pad 2: D+5V_ -> D+5V
- CN6 pad 21: unconnected-(CN6-Pad21) -> AGND
- CN6 pad 22: PE_GND -> AGND
- D17 pad 2: Net-(D1-K) -> Net-(D17-K)
- D19 pad 2: Net-(D3-K) -> Net-(D19-K)
- D21 pad 2: Net-(D5-K) -> Net-(D21-K)
- D23 pad 2: Net-(D7-K) -> Net-(D23-K)
- D25 pad 1: D+5V_ -> D+5V
- D26 pad 1: D+5V_ -> D+5V
- D27 pad 1: D+5V_ -> D+5V
- D30 pad 1: D+5V_ -> D+5V
- D31 pad 1: D+5V_ -> D+5V
- D31 pad 2: D+5V -> Header-D+5V
- DSUB1 pad 1: D+5V_ -> D+5V
- DSUB1 pad 16: unconnected-(DSUB1-Pad16) -> PE_GND
- DSUB2 pad 1: D+5V_ -> D+5V
- DSUB2 pad 10: Net-(DSUB2-MH1) -> PE_GND
- DSUB2 pad 11: Net-(DSUB2-MH1) -> PE_GND
- DSUB3 pad 1: D+5V_ -> D+5V
- DSUB3 pad 10: Net-(DSUB3-MH1) -> PE_GND
- DSUB3 pad 11: Net-(DSUB3-MH1) -> PE_GND
- DSUB4 pad 1: D+5V_ -> D+5V
- DSUB4 pad 10: Net-(DSUB4-MH1) -> PE_GND
- DSUB4 pad 11: Net-(DSUB4-MH1) -> PE_GND
- DSUB5 pad 1: D+5V_ -> D+5V
- DSUB5 pad 10: Net-(DSUB5-MH1) -> PE_GND
- DSUB5 pad 11: Net-(DSUB5-MH1) -> PE_GND
- J3 pad 10: D+5V -> Header-D+5V
- J3 pad 7: D+5V -> Header-D+5V
- J3 pad 8: D+5V -> Header-D+5V
- J3 pad 9: D+5V -> Header-D+5V
- J5 pad 1: +3.3V -> VDD
- J5 pad 2: +3.3V -> VDD
- J6 pad 1: +3.3V -> VDD
- J6 pad 2: +3.3V -> VDD
- J7 pad 11: D+5V_ -> D+5V
- J7 pad 12: D+5V_ -> D+5V
- J7 pad 13: D+5V_ -> D+5V
- J7 pad 14: D+5V_ -> D+5V
- J7 pad 17: unconnected-(J7-Pad17) -> PE_GND
- J7 pad 18: unconnected-(J7-Pad18) -> PE_GND
- Q1 pad 14: D+5V_ -> D+5V
- Q10 pad 4: D+5V_ -> D+5V
- Q11 pad 8: D+5V_ -> D+5V
- Q12 pad 8: D+5V_ -> D+5V
- Q13 pad 14: D+5V_ -> D+5V
- Q14 pad 4: D+5V_ -> D+5V
- Q15 pad 8: D+5V_ -> D+5V
- Q16 pad 8: D+5V_ -> D+5V
- Q19 pad 16: D+5V_ -> D+5V
- Q2 pad 4: D+5V_ -> D+5V
- Q20 pad 16: D+5V_ -> D+5V
- Q21 pad 8: D+5V_ -> D+5V
- Q23 pad 8: D+5V_ -> D+5V
- Q26 pad 1: Net-(D2-K) -> Net-(D17-K)
- Q26 pad 19: Net-(D1-K) -> Net-(D17-K)
- Q26 pad 20: D+5V_ -> D+5V
- Q29 pad 1: Net-(D4-K) -> Net-(D19-K)
- Q29 pad 19: Net-(D3-K) -> Net-(D19-K)
- Q29 pad 20: D+5V_ -> D+5V
- Q3 pad 8: D+5V_ -> D+5V
- Q32 pad 1: Net-(D6-K) -> Net-(D21-K)
- Q32 pad 19: Net-(D5-K) -> Net-(D21-K)
- Q32 pad 20: D+5V_ -> D+5V
- Q35 pad 1: Net-(D8-K) -> Net-(D23-K)
- Q35 pad 19: Net-(D7-K) -> Net-(D23-K)
- Q35 pad 20: D+5V_ -> D+5V
- Q4 pad 8: D+5V_ -> D+5V
- Q42 pad 3: D+5V_ -> D+5V
- Q43 pad 3: D+5V_ -> D+5V
- Q44 pad 7: D+5V_ -> D+5V
- Q44 pad 8: D+5V_ -> D+5V
- Q45 pad 2: +3.3V -> VDD
- Q45 pad 3: D+5V_ -> D+5V
- Q48 pad 5: D+5V_ -> D+5V
- Q5 pad 14: D+5V_ -> D+5V
- Q6 pad 4: D+5V_ -> D+5V
- Q7 pad 8: D+5V_ -> D+5V
- Q8 pad 8: D+5V_ -> D+5V
- Q9 pad 14: D+5V_ -> D+5V
- R167 pad 1: D+5V_ -> D+5V
- R17 pad 1: D+5V_ -> D+5V
- R174 pad 2: D+5V_ -> D+5V
- R177 pad 1: D+5V_ -> D+5V
- R184 pad 2: D+5V_ -> D+5V
- R20 pad 2: D+5V_ -> D+5V
- R206 pad 1: Net-(D4-K) -> /DSP_PWM1_~{FAULT}
- R206 pad 2: AGND -> Net-(Q28-A)
- R21 pad 2: D+5V_ -> D+5V
- R220 pad 1: Net-(D6-K) -> Net-(Q30-B)
- R220 pad 2: AGND -> /DSP_PWM1_~{FAULT}
- R222 pad 1: Net-(D5-K) -> Net-(Q30-C)
- R222 pad 2: AGND -> Net-(D20-K)
- R291 pad 2: D+5V_ -> D+5V
- R293 pad 2: D+5V_ -> D+5V
- R295 pad 2: D+5V_ -> D+5V
- R31 pad 2: D+5V_ -> D+5V
- R40 pad 1: D+5V_ -> D+5V
- R43 pad 2: D+5V_ -> D+5V
- R44 pad 2: D+5V_ -> D+5V
- R54 pad 2: D+5V_ -> D+5V
- R63 pad 1: D+5V_ -> D+5V
- R66 pad 2: D+5V_ -> D+5V
- R67 pad 2: D+5V_ -> D+5V
- R77 pad 2: D+5V_ -> D+5V
- R8 pad 2: D+5V_ -> D+5V
- R86 pad 1: D+5V_ -> D+5V
- R89 pad 2: D+5V_ -> D+5V
- R90 pad 2: D+5V_ -> D+5V
- U1 pad 1: D+5V_ -> D+5V
- U2 pad 1: Net-(TP1-Pad1) -> unconnected-(U2-3.3V-Pad1)
- U2 pad 11: D+5V_ -> D+5V
- U2 pad 12: D+5V_ -> D+5V
- U2 pad 13: D+5V_ -> D+5V
- U2 pad 14: D+5V_ -> D+5V
- U2 pad 15: D+5V_ -> D+5V
- U2 pad 16: D+5V_ -> D+5V
- U2 pad 2: Net-(TP2-Pad1) -> unconnected-(U2-3.3V-Pad2)
- U2 pad 3: Net-(TP1-Pad1) -> unconnected-(U2-3.3V-Pad3)
- U2 pad 4: Net-(TP2-Pad1) -> unconnected-(U2-3.3V-Pad4)
- U2 pad 5: Net-(TP1-Pad1) -> unconnected-(U2-3.3V-Pad5)
- U2 pad 6: Net-(TP2-Pad1) -> unconnected-(U2-3.3V-Pad6)
- U3 pad 1: D+5V_ -> D+5V
- U3 pad 25: VDD -> unconnected-(U3-3.3V-Pad25)
- U3 pad 26: VDD -> unconnected-(U3-3.3V-Pad26)
- U3 pad 27: VDD -> unconnected-(U3-3.3V-Pad27)
- U3 pad 28: VDD -> unconnected-(U3-3.3V-Pad28)
- U3 pad 29: D+5V_ -> D+5V
- U3 pad 30: D+5V_ -> D+5V
- U3 pad 31: D+5V_ -> D+5V
- U3 pad 32: D+5V_ -> D+5V
- U4 pad 40: D+5V_ -> D+5V
- U5 pad 1: D+5V_ -> D+5V
- U5 pad 40: D+5V_ -> D+5V
- U6 pad 1: D+5V_ -> D+5V
- U7 pad 1: /DSP-PWM11A -> AGND
- U7 pad 10: /MSDAA -> /MSCLA
- U7 pad 11: /DSP_Discharge1_EN -> /ADC_DO_W_3
- U7 pad 12: /ADC_DO_W_3 -> /DSP_Discharge1_EN
- U7 pad 13: /DSP_B_CAN_RX -> /MCU_EnDO_B1
- U7 pad 14: /MCU_EnDO_B1 -> /DSP_B_CAN_RX
- U7 pad 15: /DSP_B_CAN_EN -> /MCU_EnDI_B1
- U7 pad 16: /MCU_EnDI_B1 -> /DSP_B_CAN_EN
- U7 pad 17: /DSP_B_CAN_TX -> AGND
- U7 pad 18: AGND -> /DSP_B_CAN_TX
- U7 pad 19: /IPM_Temperature4 -> /DSP_Temperature1
- U7 pad 2: AGND -> /DSP-PWM11A
- U7 pad 20: /IPM_Temperature1 -> /DSP_Temperature4
- U7 pad 21: /IPM_Temperature3 -> /DSP_Temperature2
- U7 pad 22: /IPM_Temperature2 -> /DSP_Temperature3
- U7 pad 23: unconnected-(U7-AD14-Pad23) -> /DSP_VDC_BUS2
- U7 pad 24: /IPM_VDC_BUS2 -> unconnected-(U7-A3-Pad24)
- U7 pad 25: unconnected-(U7-AD15-Pad25) -> /DSP_VDC_BUS1
- U7 pad 26: /IPM_VDC_BUS1 -> unconnected-(U7-A2-Pad26)
- U7 pad 27: /IPM_VDC_BUS3 -> /DSP_VDC_BUS4
- U7 pad 28: /IPM_VDC_BUS4 -> /DSP_VDC_BUS3
- U7 pad 29: /DSP-PWM7B -> AGND
- U7 pad 3: /DSP-PWM11B -> /DSP-PWM7A
- U7 pad 30: AGND -> /DSP-PWM7B
- U7 pad 4: /DSP-PWM7A -> /DSP-PWM11B
- U7 pad 5: /DSP_A_CAN_RX -> /DSP_A_CAN_TX
- U7 pad 6: /DSP_A_CAN_TX -> /DSP_A_CAN_RX
- U7 pad 7: /DSP-PWM2B -> /DSP_A_CAN_EN
- U7 pad 8: /DSP_A_CAN_EN -> /DSP-PWM2B
- U7 pad 9: /MSCLA -> /MSDAA
Routing:
- net D+5V: track 0.00 -> 1568.3 mm, vias 0 -> 94
- net VDD: track 174.1 -> 1285.9 mm, vias 17 -> 97
- net AGND: track 39.1 -> 668.0 mm, vias 24 -> 1585
- net /DSP_Temperature1: track 0.00 -> 166.4 mm, vias 0 -> 1
- net /IPM_Temperature1: track 160.9 -> 0.00 mm, vias 1 -> 0
- net /DSP_VDC_BUS1: track 0.00 -> 155.7 mm, vias 0 -> 1
- net /IPM_VDC_BUS1: track 154.3 -> 0.00 mm, vias 1 -> 0
- net D+5V_: track 137.4 -> 0.00 mm, vias 8 -> 0
- net /DSP_VDC_BUS2: track 0.00 -> 129.0 mm
- net /DSP_Temperature2: track 0.00 -> 125.5 mm
- net /IPM_VDC_BUS2: track 114.0 -> 0.00 mm
- net /IPM_Temperature2: track 109.5 -> 0.00 mm
- net /ADC_CLK_X2: track 180.2 -> 263.8 mm, vias 1 -> 3
- net /IPM_VDC_BUS3: track 62.0 -> 0.00 mm
- net /DSP_VDC_BUS3: track 0.00 -> 61.1 mm
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- added copper zone on B.Cu, net D+5V
- added copper zone on F.Cu, net D+5V
- added copper zone on F.Cu, net Header-D+5V
- added copper zone on B.Cu, net VDD
- added copper zone on F.Cu, net VDD
Other:
- board text added: "+5V"
- board text added: "A:Power_In"
- board text added: "B:Power_In"
- board text added: "CK"
- board text added: "CLK"
- board text added: "D0"
- board text added: "DATA"
- board text added: "GND"
- board text added: "MI"
- board text added: "MO"
- board text added: "NC"
- board text added: "PE"
- board text added: "RX"
- board text added: "STE"
- board text added: "TX"
- board text added: "V-CUT"
- board text added: "VDD"
- board text added: "X X"
- board text added: "→"
