File: SlaveDesignFiles/sheet1.kicad_sch (KiCad schematic)
At the start: 143 parts, among them CN7 DB141V-2.54-6P, CN8 DB141V-2.54-6P, J1 Conn_02x02_Counter_Clockwise, J2 Conn_02x02_Counter_Clockwise, J3 2.54-2*5, J4 2.54-2*5, J5 2.54-2*5, J6 2.54-2*5, J7 PM2.54-2*10, J8 2.54-2*5, M1 Conn_01x01_Socket, M2 Conn_01x01_Socket, M3 Conn_01x01_Socket, M4 Conn_01x01_Socket, M5 Conn_01x01_Socket, M6 Conn_01x01_Socket, M7 Conn_01x01_Socket, M8 Conn_01x01_Socket, Q37 FMMT618TA, Q38 FMMT618TA, Q39 FMMT618TA, Q40 SN74LVC14APWRG4, Q41 FMMT618TA, Q42 TPT1042VQ-SO1R-S, Q43 TPT1042VQ-SO1R-S, Q44 CP2102N-A02-GQFN28R, Q45 AMS1117-3.3, Q46 TYPEC-304-ACP16, Q47 AT24C16C-SSHM-T, Q48 SRV05-4HTG, U1 X1321FVS-2X20-C43D48, U2 X1321FVS-2X20-C43D48, U3 X1321FVS-2X20-C43D48, U4 X1321FVS-2X20-C43D48, U5 X1321FVS-2X20-C43D48, U6 X1321FVS-2X20-C43D48, U7 PM254-2-15-Z-8.5, X1 20MHz, X2 20MHz

Commit message: First version
Parts:
- removed TP1, TP2: TestPoint, TestPoint:TestPoint_Loop_D2.60mm_Drill1.4mm_Beaded, symbol Connector:TestPoint
- added ref1, ref2, ref3, ref4: Conn_01x01_Socket, 1mmlab_footprint:Mark_TH_3mm, symbol Connector:Conn_01x01_Socket
- added ref10, ref11, ref12, ref13, ref14, ref15, ref16, ref17, ref18, ref19, ref20, ref5, ref6, ref7, ref8, ref9: Conn_01x01_Socket, 1mmlab_footprint:Mark_SMD, symbol Connector:Conn_01x01_Socket
Connections:
- net ADC_DO_W_3: now also U7.11 (P27); no longer U7.12 (P26)
- net AGND: now also U7.1 (P20), U7.17 (P8), U7.29 (P13); no longer U7.18 (GND), U7.2 (GND), U7.30 (GND)
- net DSP-PWM11A: now also U7.2 (GND); no longer U7.1 (P20)
- net DSP-PWM11B: now also U7.4 (P12); no longer U7.3 (P21)
- net DSP-PWM2B: now also U7.8 (P2); no longer U7.7 (P3)
- net DSP-PWM7A: now also U7.3 (P21); no longer U7.4 (P12)
- net DSP-PWM7B: now also U7.30 (GND); no longer U7.29 (P13)
- net DSP_A_CAN_EN: now also U7.7 (P3); no longer U7.8 (P2)
- net DSP_A_CAN_RX: now also U7.6 (P4); no longer U7.5 (P5)
- net DSP_A_CAN_TX: now also U7.5 (P5); no longer U7.6 (P4)
- net DSP_B_CAN_EN: now also U7.16 (P24); no longer U7.15 (P9)
- net DSP_B_CAN_RX: now also U7.14 (P25); no longer U7.13 (P10)
- net DSP_B_CAN_TX: now also U7.18 (GND); no longer U7.17 (P8)
- net DSP_Discharge1_EN: now also U7.12 (P26); no longer U7.11 (P27)
- net DSP_Temperature1: now also U7.19 (C3); no longer U7.20 (B4)
- net DSP_Temperature2: now also U7.21 (C2); no longer U7.22 (B5)
- net DSP_Temperature3: now also U7.22 (B5); no longer U7.21 (C2)
- net DSP_Temperature4: now also U7.20 (B4); no longer U7.19 (C3)
- net DSP_VDC_BUS1: now also U7.25 (AD15); no longer U7.26 (A2)
- net DSP_VDC_BUS2: now also U7.23 (AD14); no longer U7.24 (A3)
- net DSP_VDC_BUS3: now also U7.28 (B3); no longer U7.27 (B2)
- net DSP_VDC_BUS4: now also U7.27 (B2); no longer U7.28 (B3)
- net MCU_EnDI_B1: now also U7.15 (P9); no longer U7.16 (P24)
- net MCU_EnDO_B1: now also U7.13 (P10); no longer U7.14 (P25)
- net MSCLA: now also U7.10 (P0); no longer U7.9 (P1)
- net MSDAA: now also U7.9 (P1); no longer U7.10 (P0)
- net PE_GND: now also DSUB1.16, DSUB2.10 (MH1), DSUB2.11 (MH2), DSUB3.10 (MH1), DSUB3.11 (MH2), DSUB4.10 (MH1), DSUB4.11 (MH2), DSUB5.10 (MH1), DSUB5.11 (MH2), J7.17, J7.18; no longer Q46.EP
- now unconnected: U2.1 (3.3V), U2.2 (3.3V), U2.3 (3.3V), U2.4 (3.3V), U2.5 (3.3V), U2.6 (3.3V)
- no-connect marks 97 -> 101
Other:
- note added: "PE螺丝孔"
- note added: "测试点"
