File: SlaveDesignFiles/FourInOne388_V01.kicad_pcb (KiCad board)
At the start: 4 copper layers, 216 x 144 mm, 616 parts, among them CN1 DB141V-2.54-6P, CN2 DB141V-2.54-6P, CN3 X3025WVS-2*10D-LPSW, CN4 X3025WVS-2*10D-LPSW, CN5 X3025WVS-2*10D-LPSW, CN6 X3025WVS-2*10D-LPSW, CN7 DB141V-2.54-6P, CN8 DB141V-2.54-6P, J1 Conn_02x02_Counter_Clockwise, J2 Conn_02x02_Counter_Clockwise, J3 2.54-2*5, J4 2.54-2*5, J5 2.54-2*5, J6 2.54-2*5, J7 PM2.54-2*10, J8 2.54-2*5, M1 Conn_01x01_Socket, M2 Conn_01x01_Socket, M3 Conn_01x01_Socket, M4 Conn_01x01_Socket, M5 Conn_01x01_Socket, M6 Conn_01x01_Socket, M7 Conn_01x01_Socket, M8 Conn_01x01_Socket, Q1 TXB0104PWR, Q10 TPS27082LDDCR, Q11 TPT75176B-SO1R, Q12 TPT75176B-SO1R, Q13 TXB0104PWR, Q14 TPS27082LDDCR, Q15 TPT75176B-SO1R, Q16 TPT75176B-SO1R, Q17 DP83822IRHBR, Q18 DP83822IRHBR, Q19 AM26C32CD, Q2 TPS27082LDDCR, Q20 AM26C32CD, Q21 TPT75176B-SO1R, Q22 SN74LVC1G125DCKR, Q23 TPT75176B-SO1R, Q24 SN74LVC1G125DCKR, Q25 SN74LVC1G125DCKR, Q26 SN74ACT244PWRG4, Q27 FMMT618TA, Q28 SN74LVC1G125DCKR, Q29 SN74ACT244PWRG4, Q3 TPT75176B-SO1R, Q30 FMMT618TA, Q31 SN74LVC1G125DCKR, Q32 SN74ACT244PWRG4, Q33 FMMT618TA, Q34 SN74LVC1G125DCKR, Q35 SN74ACT244PWRG4, Q36 FMMT618TA, Q37 FMMT618TA, Q38 FMMT618TA, Q39 FMMT618TA, Q4 TPT75176B-SO1R, Q40 SN74LVC14APWRG4, Q41 FMMT618TA, Q42 TPT1042VQ-SO1R-S, Q43 TPT1042VQ-SO1R-S, Q44 CP2102N-A02-GQFN28R, Q45 AMS1117-3.3, Q46 TYPEC-304-ACP16, Q47 AT24C16C-SSHM-T, Q48 SRV05-4HTG, Q5 TXB0104PWR, Q6 TPS27082LDDCR, Q7 TPT75176B-SO1R, Q8 TPT75176B-SO1R, Q9 TXB0104PWR, U1 X1321FVS-2X20-C43D48, U2 X1321FVS-2X20-C43D48, U3 X1321FVS-2X20-C43D48, U4 X1321FVS-2X20-C43D48, U5 X1321FVS-2X20-C43D48, U6 X1321FVS-2X20-C43D48, U7 PM254-2-15-Z-8.5, X1 20MHz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

Commit message: Fix the pin axial symmetry bug
Connections:
- U7 pad 1: AGND -> /DSP-PWM11A
- U7 pad 10: /MSCLA -> /MSDAA
- U7 pad 11: /ADC_DO_W_3 -> /DSP_Discharge1_EN
- U7 pad 12: /DSP_Discharge1_EN -> /ADC_DO_W_3
- U7 pad 13: /MCU_EnDO_B1 -> /DSP_B_CAN_RX
- U7 pad 14: /DSP_B_CAN_RX -> /MCU_EnDO_B1
- U7 pad 15: /MCU_EnDI_B1 -> /DSP_B_CAN_EN
- U7 pad 16: /DSP_B_CAN_EN -> /MCU_EnDI_B1
- U7 pad 17: AGND -> /DSP_B_CAN_TX
- U7 pad 18: /DSP_B_CAN_TX -> AGND
- U7 pad 19: /DSP_Temperature1 -> /DSP_Temperature4
- U7 pad 2: /DSP-PWM11A -> AGND
- U7 pad 20: /DSP_Temperature4 -> /DSP_Temperature1
- U7 pad 21: /DSP_Temperature2 -> /DSP_Temperature3
- U7 pad 22: /DSP_Temperature3 -> /DSP_Temperature2
- U7 pad 23: /DSP_VDC_BUS2 -> unconnected-(U7-AD14-Pad23)
- U7 pad 24: unconnected-(U7-A3-Pad24) -> /DSP_VDC_BUS2
- U7 pad 25: /DSP_VDC_BUS1 -> unconnected-(U7-AD15-Pad25)
- U7 pad 26: unconnected-(U7-A2-Pad26) -> /DSP_VDC_BUS1
- U7 pad 27: /DSP_VDC_BUS4 -> /DSP_VDC_BUS3
- U7 pad 28: /DSP_VDC_BUS3 -> /DSP_VDC_BUS4
- U7 pad 29: AGND -> /DSP-PWM7B
- U7 pad 3: /DSP-PWM7A -> /DSP-PWM11B
- U7 pad 30: /DSP-PWM7B -> AGND
- U7 pad 4: /DSP-PWM11B -> /DSP-PWM7A
- U7 pad 5: /DSP_A_CAN_TX -> /DSP_A_CAN_RX
- U7 pad 6: /DSP_A_CAN_RX -> /DSP_A_CAN_TX
- U7 pad 7: /DSP_A_CAN_EN -> /DSP-PWM2B
- U7 pad 8: /DSP-PWM2B -> /DSP_A_CAN_EN
- U7 pad 9: /MSDAA -> /MSCLA
Routing:
- net /MSDAA: track 108.9 -> 117.4 mm, vias 1 -> 2
- net /DSP_VDC_BUS1: track 155.7 -> 160.3 mm
- net /DSP_PWM4~{_ENABL}E: track 106.4 -> 110.6 mm
- net /DSP-PWM11B: track 41.6 -> 37.5 mm
- net /DSP_Temperature2: track 125.5 -> 121.5 mm
- net /DSP_VDC_BUS2: track 129.0 -> 125.1 mm
- net /DSP_A_CAN_EN: track 26.4 -> 30.4 mm, vias 0 -> 1
- net /DSP_Discharge1_EN: track 124.2 -> 127.7 mm
- net /DSP-PWM2B: track 109.8 -> 113.3 mm
- net /DSP_A_CAN_TX: track 25.7 -> 29.1 mm, vias 0 -> 1
- net /MQEP1A: track 125.6 -> 122.5 mm
- net /MQEP1B: track 131.3 -> 128.1 mm
- net /DSP-PWM11A: track 44.8 -> 42.1 mm
- net /DSP_Temperature4: track 46.3 -> 43.7 mm
- net /DSP_VDC_BUS4: track 53.4 -> 56.0 mm
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