File: SlaveDesignFiles/26c32.kicad_sch (KiCad schematic)
At the start: 35 parts, among them Q19 AM26C32CD

Commit message: 28388d直接在底板上
Parts:
- removed C73, C74, C75, C76, C77, C78, C79, C80, C81: 100pF/50V, Capacitor_SMD:C_0603_1608Metric, symbol sheet1-altium-import:CAP_1
- removed C82: 0.1uF/50V, Capacitor_SMD:C_0603_1608Metric, symbol sheet1-altium-import:CAP_2
- removed D10, D11, D9: SDT23C712L02_C5197393, Lib2ic:SOT-23-3_L2.9-W1.3-P1.90-LS2.4-BR, symbol sheet1-altium-import:SDT23C712L02_C5197393
- removed L10, L9: AMCW3225P-2-242T, Lib_sheet_10:FILTER-SMD_4P-L3.2-W2.5-BL_WCM3225XXXX, symbol sheet1-altium-import:AMCW3225P-2-242T
- removed R131, R132, R133: 2.2K/1%, Resistor_SMD:R_0603_1608Metric, symbol sheet1-altium-import:RES_1
- removed R134, R135, R136, R137, R138, R139: 47R/1%, Lib_sheet_10:R_0603_1608Metric, symbol sheet1-altium-import:RES_2
- removed R140, R141, R142, R143, R144, R145: 5.1K/1%, Resistor_SMD:R_0603_1608Metric, symbol sheet1-altium-import:RES_3
- removed R146, R147, R148: 62R/1%, Resistor_SMD:R_0603_1608Metric, symbol sheet1-altium-import:RES_4
- added C184, C185, C186, C187, C188, C189, C190, C191, C192: 100pF/50V, Capacitor_SMD:C_0603_1608Metric, symbol sheet1-altium-import:CAP_1
- added C193: 0.1uF/50V, Capacitor_SMD:C_0603_1608Metric, symbol sheet1-altium-import:CAP_2
- added D36, D37, D38: SDT23C712L02_C5197393, Lib2ic:SOT-23-3_L2.9-W1.3-P1.90-LS2.4-BR, symbol sheet1-altium-import:SDT23C712L02_C5197393
- added L16, L17: AMCW3225P-2-242T, Lib_sheet_10:FILTER-SMD_4P-L3.2-W2.5-BL_WCM3225XXXX, symbol sheet1-altium-import:AMCW3225P-2-242T
- added R291, R292, R293: 2.2K/1%, Resistor_SMD:R_0603_1608Metric, symbol sheet1-altium-import:RES_1
- added R294, R295, R296, R297, R298, R299: 47R/1%, Lib_sheet_10:R_0603_1608Metric, symbol sheet1-altium-import:RES_2
- added R300, R301, R302, R303, R304, R305: 5.1K/1%, Resistor_SMD:R_0603_1608Metric, symbol sheet1-altium-import:RES_3
- added R306, R307, R308: 62R/1%, Resistor_SMD:R_0603_1608Metric, symbol sheet1-altium-import:RES_4
- renumbered L11 to L18, Q19 to Q47
Connections:
- net 1A: now also L16.4
- net 1B: now also L16.1
- net 1Y: now also R306.2
- net 2A: now also L17.4
- net 2B: now also L17.1
- net 2Y: now also R307.2
- net 3Y: now also R308.1
- net AGND: now also C184.2, C185.2, C186.2, C190.2, C191.2, C192.2, C193.2, D36.3, D37.3, D38.3, R300.1, R301.1, R302.1, R303.1, R304.1, R305.1
- net D+5V: now also C193.1
- net at Q47.7 (2B): now also R297.2, R301.2
- net at L18.3: now also C186.1, C189.2, D38.2, R293.1, R299.1
- net at Q47.10 (3A): now also R299.2, R302.2
- net at Q47.6 (2A): now also R296.2, R304.2
- net at Q47.1 (1B): now also R294.2, R303.2
- net at Q47.9 (3B): now also R298.2, R305.2
- net at Q47.11 (3Y): now also R308.2
- net at L18.2: now also C189.1, C192.1, D38.1, R293.2, R298.1
- net at Q47.5 (2Y): now also R307.1
- net at Q47.2 (1A): now also R295.2, R300.2
- net at Q47.3 (1Y): now also R306.1
- new net: C188.1, C191.1, D37.2, L17.3, R292.2, R296.1
- new net: C184.1, C187.2, D36.2, L16.3, R291.1, R294.1
- new net: C187.1, C190.1, D36.1, L16.2, R291.2, R295.1
- new net: C185.1, C188.2, D37.1, L17.2, R292.1, R297.1
Other:
- moved on the sheet: L18, Q47
