File: SlaveDesignFiles/ETHERCAT.kicad_sch (KiCad schematic)
At the start: 33 parts, among them Q17 DP83822IRHBR

Commit message: 28388d直接在底板上
Parts:
- removed C49: 0.01uF/50V, Capacitor_SMD:C_0603_1608Metric, symbol sheet1-altium-import:CAP_1
- removed C50: 0.1uF/50V, Capacitor_SMD:C_0603_1608Metric, symbol sheet1-altium-import:CAP_2
- added C78: 0.01uF/50V, Capacitor_SMD:C_0603_1608Metric, symbol sheet1-altium-import:CAP_1
- added C79, C90, C92: 0.1uF/50V, Capacitor_SMD:C_0603_1608Metric, symbol sheet1-altium-import:CAP_2
- added C91, C93: 1uF/16V, Capacitor_SMD:C_0603_1608Metric, symbol sheet1-altium-import:CAP_3
- R80: renamed from R104; value 2.2K/1% -> 10.0K/1%
- renumbered C51 to C80, C52 to C81, C53 to C82, C54 to C83, C55 to C84, C56 to C85, C57 to C86, C58 to C87, C59 to C88, C60 to C89, Q17 to Q13, R93 to R69, R94 to R70, R95 to R71, R96 to R72, R97 to R73, R98 to R74, R99 to R75, R100 to R76, R101 to R77, R102 to R78, R103 to R79, R105 to R81, R106 to R82, R107 to R83, R108 to R84, R109 to R85, R110 to R86, R111 to R87
Connections:
- net VDD is gone; now on net +3V3D_DSP: C80.2, C81.2, C82.2, C83.1, C84.2, C85.2, C86.1, C87.2, C88.1, C89.2, Q13.14 (AVD), Q13.21 (VDDIO), R75.2, R76.2, R78.2, R79.1, R80.1, R81.2, R82.2, R83.2, R84.2, R85.2, R86.1, R87.1
- net at Q13.29 (COL/GPIO2): now also R74.1; no longer R74.2
- net +3V3D_DSP: now reaches RJ1.1.P3 (RCT)
- net +3V3D_DSP: now also R74.2, RJ1.1.P4 (TCT), C78.2, C79.1, C90.1, C91.2, C92.1, C93.2
- net AGND renamed GND
- net GND: now also C78.1, C79.2, C90.2, C91.1, C92.2, C93.1; no longer R74.1
- no-connect marks 6 -> 4
Other:
- moved on the sheet: C80, C81, C82, C83, C84, C85, C86, C87, C88, C89, Q13, R69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
