File: SlaveDesignFiles/ETHERCAT2.kicad_sch (KiCad schematic)
At the start: 33 parts, among them Q18 DP83822IRHBR

Commit message: 28388d直接在底板上
Parts:
- added C106, C108: 0.1uF/50V, Capacitor_SMD:C_0603_1608Metric, symbol sheet1-altium-import:CAP_2
- added C107, C109: 1uF/16V, Capacitor_SMD:C_0603_1608Metric, symbol sheet1-altium-import:CAP_3
- R99: renamed from R123; value 2.2K/1% -> 10K/1%
- renumbered C67 to C100, C68 to C101, C69 to C102, C70 to C103, C71 to C104, C72 to C105, C61 to C94, C62 to C95, C63 to C96, C64 to C97, C65 to C98, C66 to C99, Q18 to Q14, R124 to R100, R125 to R101, R126 to R102, R127 to R103, R128 to R104, R129 to R105, R130 to R106, R112 to R88, R113 to R89, R114 to R90, R115 to R91, R116 to R92, R117 to R93, R118 to R94, R119 to R95, R120 to R96, R121 to R97, R122 to R98
Connections:
- net VDD is gone; now on net +3V3D_DSP: C100.2, C101.2, C102.1, C103.2, C104.1, C105.2, C94.2, C95.1, C96.2, C97.2, C98.2, C99.1, Q14.14 (AVD), Q14.21 (VDDIO), R100.2, R101.2, R102.2, R103.2, R104.2, R105.1, R106.1, R94.2, R95.2, R97.2, R98.1, R99.1
- net at Q14.29 (COL/GPIO2): now also R93.1; no longer R93.2
- net +3V3D_DSP: now reaches RJ1.1.3 (RCT)
- net +3V3D_DSP: now also R93.2, RJ1.1.4 (TCT), C106.1, C107.2, C108.1, C109.2
- net AGND renamed GND
- net GND: now also C106.2, C107.1, C108.2, C109.1; no longer R93.1
- no-connect marks 6 -> 4
Other:
- moved on the sheet: C100, C101, C102, C103, C104, C105, C94, C95, C96, C97, C98, C99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
