File: SlaveDesignFiles/H485.kicad_sch (KiCad schematic)
At the start: 22 parts, among them CN1 DB141V-2.54-6P, Q21 TPT75176B-SO1R, Q22 SN74LVC1G125DCKR

Commit message: 28388d直接在底板上
Parts:
- removed C93, C95: 100pF/50V, Capacitor_SMD:C_0603_1608Metric, symbol sheet1-altium-import:CAP_1
- removed C94: 15pF/50V, Capacitor_SMD:C_0603_1608Metric, symbol sheet1-altium-import:CAP
- removed C96: 0.1uF/50V, Capacitor_SMD:C_0603_1608Metric, symbol sheet1-altium-import:CAP_2
- removed C97: 0.01uF/50V, Capacitor_SMD:C_0603_1608Metric, symbol sheet1-altium-import:CAP_1
- removed C98, C99: 330pF/50V, Capacitor_SMD:C_0603_1608Metric, symbol sheet1-altium-import:CAP_1
- added C170, C172: 100pF/50V, Capacitor_SMD:C_0603_1608Metric, symbol sheet1-altium-import:CAP_1
- added C171: 15pF/50V, Capacitor_SMD:C_0603_1608Metric, symbol sheet1-altium-import:CAP
- added C173: 0.1uF/50V, Capacitor_SMD:C_0603_1608Metric, symbol sheet1-altium-import:CAP_2
- added C174: 0.01uF/50V, Capacitor_SMD:C_0603_1608Metric, symbol sheet1-altium-import:CAP_1
- added C175, C176: 330pF/50V, Capacitor_SMD:C_0603_1608Metric, symbol sheet1-altium-import:CAP_1
- renumbered CN1 to CN7, D15 to D34, L15 to L14, Q21 to Q43, Q22 to Q44, R167 to R271, R168 to R272, R169 to R273, R170 to R274, R171 to R275, R172 to R276, R173 to R277, R174 to R278, R175 to R279, R176 to R280
Connections:
- net AGND: now also C170.2, C171.1, C172.2, C173.2, C174.1, C175.2, C176.2
- net D+5V: now also C173.1
- net VDD: now also C174.2
- net at Q43.2 (RE#), Q43.3 (DE), R272.1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: now also C172.1
- net at D34.1, L14.4, Q43.7 (B)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: now also C175.1
- net at D34.2, L14.1, Q43.6 (A)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: now also C176.1
- net at Q43.4 (D), R273.1, R274.2: now also C170.1
- net at Q44.2 (A), R275.2: now also C171.2
Other:
- moved on the sheet: CN7, D34, L14, Q43, Q44, R271, R272, R273, R274, R275, R276, R277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
