File: SlaveDesignFiles/IPM.kicad_sch (KiCad schematic)
At the start: 27 parts, among them CN3 X3025WVS-2*10D-LPSW, Q25 SN74LVC1G125DCKR, Q26 SN74ACT244PWRG4, Q27 FMMT618TA

Commit message: First version
Connections:
- net PE_GND is gone; now on net AGND: CN3.22
- net AGND: now also CN3.21
- no-connect marks 3 -> 2

Commit message: 28388d直接在底板上
Parts:
- removed C107: 15pF/50V, Capacitor_SMD:C_0603_1608Metric, symbol sheet1-altium-import:CAP
- removed C108: 0.01uF/50V, Capacitor_SMD:C_0603_1608Metric, symbol sheet1-altium-import:CAP_1
- removed C109: 0.1uF/50V, Capacitor_SMD:C_0603_1608Metric, symbol sheet1-altium-import:CAP_2
- added C158: 15pF/50V, Capacitor_SMD:C_0603_1608Metric, symbol sheet1-altium-import:CAP
- added C159: 0.01uF/50V, Capacitor_SMD:C_0603_1608Metric, symbol sheet1-altium-import:CAP_1
- added C160: 0.1uF/50V, Capacitor_SMD:C_0603_1608Metric, symbol sheet1-altium-import:CAP_2
- renumbered D17 to D26, D18 to D27, Q25 to Q31, Q26 to Q32, Q27 to Q33, R187 to R199, R188 to R200, R189 to R201, R190 to R202, R191 to R203, R192 to R204, R193 to R205, R194 to R206, R195 to R207, R196 to R208, R197 to R209, R198 to R210, R199 to R211, R200 to R212, R201 to R213, R202 to R214, R203 to R215, R204 to R216
Connections:
- net AGND: now also C158.1, C159.1, C160.2
- net D+5V: now also C160.1
- net VDD: now also C159.2
- net at Q31.2 (A), R200.2: now also C158.2
Other:
- moved on the sheet: CN3, D26, D27, Q31, Q32, Q33, R199, R200, R201, R202, R203, R204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
