File: 28388BGA/26c32.kicad_sch (KiCad schematic)
At the start: 35 parts, among them Q47 AM26C32CD

Commit message: 修复AGND BUG
Connections:
- net AGND renamed GND
Changed lines of the file:
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@@
 		(on_board yes)
 		(dnp no)
-		(property "Reference" "#PWR0473"
-			(at 106.68 111.76 0)
+		(property "Reference" "#PWR473"
+			(at 106.68 118.11 0)
 			(effects
 				(font
@@
 			)
 		)
-		(property "Value" "AGND"
-			(at 106.68 118.11 0)
+		(property "Value" "GND"
+			(at 106.68 115.57 0)
 			(effects
 				(font
 					(size 1.27 1.27)
 				)
-				(hide yes)
 			)
 		)
@@
 			(project "28388bga"
 				(path "/88c87a56-bf0e-49aa-812f-d0846700c8ff/42063a57-6d21-4a6b-b607-9c1cfdab080d"
-					(reference "#PWR0529")
+					(reference "#PWR529")
 					(unit 1)
 				)
 				(path "/88c87a56-bf0e-49aa-812f-d0846700c8ff/7fd0243d-018a-444a-b841-9493ffd32c74"
-					(reference "#PWR0473")
+					(reference "#PWR473")
 					(unit 1)
 				)
 				(path "/88c87a56-bf0e-49aa-812f-d0846700c8ff/df82ad4c-ed56-4ee7-81c5-26093527e3af"
-					(reference "#PWR0481")
+					(reference "#PWR481")
 					(unit 1)
 				)
@@
 		(on_board yes)
 		(dnp no)
-		(property "Reference" "#PWR0477"
-			(at 205.74 102.87 0)
+		(property "Reference" "#PWR477"
+			(at 205.74 109.22 0)
 			(effects
 				(font
@@
 			)
 		)
-		(property "Value" "AGND"
-			(at 205.74 109.22 0)
+		(property "Value" "GND"
+			(at 205.74 106.68 0)
 			(effects
 				(font
 					(size 1.27 1.27)
 				)
-				(hide yes)
 			)
 		)
@@
 			(project "28388bga"
 				(path "/88c87a56-bf0e-49aa-812f-d0846700c8ff/42063a57-6d21-4a6b-b607-9c1cfdab080d"
-					(reference "#PWR0533")
+					(reference "#PWR533")
 					(unit 1)
 				)
 				(path "/88c87a56-bf0e-49aa-812f-d0846700c8ff/7fd0243d-018a-444a-b841-9493ffd32c74"
-					(reference "#PWR0477")
+					(reference "#PWR477")
 					(unit 1)
 				)
 				(path "/88c87a56-bf0e-49aa-812f-d0846700c8ff/df82ad4c-ed56-4ee7-81c5-26093527e3af"
-					(reference "#PWR0485")
+					(reference "#PWR485")
 					(unit 1)
 				)
@@
 		(on_board yes)
 		(dnp no)
-		(property "Reference" "#PWR0478"
-			(at 227.33 52.07 0)
+		(property "Reference" "#PWR478"
+			(at 233.68 52.07 0)
 			(effects
 				(font
@@
 			)
 		)
-		(property "Value" "AGND"
-			(at 233.68 52.07 0)
+		(property "Value" "GND"
+			(at 231.14 52.07 0)
 			(effects
 				(font
 					(size 1.27 1.27)
 				)
-				(hide yes)
 			)
 		)
@@
 			(project "28388bga"
 				(path "/88c87a56-bf0e-49aa-812f-d0846700c8ff/42063a57-6d21-4a6b-b607-9c1cfdab080d"
-					(reference "#PWR0534")
+					(reference "#PWR534")
 					(unit 1)
 				)
 				(path "/88c87a56-bf0e-49aa-812f-d0846700c8ff/7fd0243d-018a-444a-b841-9493ffd32c74"
-					(reference "#PWR0478")
+					(reference "#PWR478")
 					(unit 1)
 				)
 				(path "/88c87a56-bf0e-49aa-812f-d0846700c8ff/df82ad4c-ed56-4ee7-81c5-26093527e3af"
-					(reference "#PWR0486")
+					(reference "#PWR486")
 					(unit 1)
 				)
@@
 		(on_board yes)
 		(dnp no)
-		(property "Reference" "#PWR0475"
-			(at 163.83 77.47 0)
+		(property "Reference" "#PWR475"
+			(at 157.48 77.47 0)
 			(effects
 				(font
@@
 			)
 		)
-		(property "Value" "AGND"
-			(at 157.48 77.47 0)
+		(property "Value" "GND"
+			(at 160.02 77.47 0)
 			(effects
 				(font
 					(size 1.27 1.27)
 				)
-				(hide yes)
 			)
 		)
@@
 			(project "28388bga"
 				(path "/88c87a56-bf0e-49aa-812f-d0846700c8ff/42063a57-6d21-4a6b-b607-9c1cfdab080d"
-					(reference "#PWR0531")
+					(reference "#PWR531")
 					(unit 1)
 				)
 				(path "/88c87a56-bf0e-49aa-812f-d0846700c8ff/7fd0243d-018a-444a-b841-9493ffd32c74"
-					(reference "#PWR0475")
+					(reference "#PWR475")
 					(unit 1)
 				)
 				(path "/88c87a56-bf0e-49aa-812f-d0846700c8ff/df82ad4c-ed56-4ee7-81c5-26093527e3af"
-					(reference "#PWR0483")
+					(reference "#PWR483")
 					(unit 1)
 				)
@@
 		(on_board yes)
 		(dnp no)
-		(property "Reference" "#PWR0479"
-			(at 227.33 77.47 0)
+		(property "Reference" "#PWR479"
+			(at 233.68 77.47 0)
 			(effects
 				(font
@@
 			)
 		)
-		(property "Value" "AGND"
-			(at 233.68 77.47 0)
+		(property "Value" "GND"
+			(at 231.14 77.47 0)
 			(effects
 				(font
 					(size 1.27 1.27)
 				)
-				(hide yes)
 			)
 		)
@@
 			(project "28388bga"
 				(path "/88c87a56-bf0e-49aa-812f-d0846700c8ff/42063a57-6d21-4a6b-b607-9c1cfdab080d"
-					(reference "#PWR0535")
+					(reference "#PWR535")
 					(unit 1)
 				)
 				(path "/88c87a56-bf0e-49aa-812f-d0846700c8ff/7fd0243d-018a-444a-b841-9493ffd32c74"
-					(reference "#PWR0479")
+					(reference "#PWR479")
 					(unit 1)
 				)
 				(path "/88c87a56-bf0e-49aa-812f-d0846700c8ff/df82ad4c-ed56-4ee7-81c5-26093527e3af"
-					(reference "#PWR0487")
+					(reference "#PWR487")
 					(unit 1)
 				)
@@
 		(on_board yes)
 		(dnp no)
-		(property "Reference" "#PWR0472"
-			(at 106.68 78.74 0)
+		(property "Reference" "#PWR472"
+			(at 106.68 85.09 0)
 			(effects
 				(font
@@
 			)
 		)
-		(property "Value" "AGND"
-			(at 106.68 85.09 0)
+		(property "Value" "GND"
+			(at 106.68 82.55 0)
 			(effects
 				(font
 					(size 1.27 1.27)
 				)
-				(hide yes)
 			)
 		)
@@
 			(project "28388bga"
 				(path "/88c87a56-bf0e-49aa-812f-d0846700c8ff/42063a57-6d21-4a6b-b607-9c1cfdab080d"
-					(reference "#PWR0528")
+					(reference "#PWR528")
 					(unit 1)
 				)
 				(path "/88c87a56-bf0e-49aa-812f-d0846700c8ff/7fd0243d-018a-444a-b841-9493ffd32c74"
-					(reference "#PWR0472")
+					(reference "#PWR472")
 					(unit 1)
 				)
 				(path "/88c87a56-bf0e-49aa-812f-d0846700c8ff/df82ad4c-ed56-4ee7-81c5-26093527e3af"
-					(reference "#PWR0480")
+					(reference "#PWR480")
 					(unit 1)
 				)
@@
 		(on_board yes)
 		(dnp no)
-		(property "Reference" "#PWR0474"
-			(at 106.68 146.05 0)
+		(property "Reference" "#PWR474"
+			(at 106.68 152.4 0)
 			(effects
 				(font
@@
 			)
 		)
-		(property "Value" "AGND"
-			(at 106.68 152.4 0)
+		(property "Value" "GND"
+			(at 106.68 149.86 0)
 			(effects
 				(font
 					(size 1.27 1.27)
 				)
-				(hide yes)
 			)
 		)
@@
 			(project "28388bga"
 				(path "/88c87a56-bf0e-49aa-812f-d0846700c8ff/42063a57-6d21-4a6b-b607-9c1cfdab080d"
-					(reference "#PWR0530")
+					(reference "#PWR530")
 					(unit 1)
 				)
 				(path "/88c87a56-bf0e-49aa-812f-d0846700c8ff/7fd0243d-018a-444a-b841-9493ffd32c74"
-					(reference "#PWR0474")
+					(reference "#PWR474")
 					(unit 1)
 				)
 				(path "/88c87a56-bf0e-49aa-812f-d0846700c8ff/df82ad4c-ed56-4ee7-81c5-26093527e3af"
-					(reference "#PWR0482")
+					(reference "#PWR482")
 					(unit 1)
 				)
