File: 28388BGA/28388bga.kicad_sch (KiCad schematic)
At the start: 223 parts, among them CN1 DB141V-2.54-6P, CN2 DB141V-2.54-6P, IC1 F28388DZWTS, IC10 TPD4E001QDBVRQ1, IC11 TPD4E001QDBVRQ1, IC2 TPS62420DRCT, IC3 TPD4E001QDBVRQ1, IC4 TPD4E001QDBVRQ1, IC5 TPD4E001QDBVRQ1, IC6 OPA4350EA_250, IC7 TPS3702CX33DDCT, IC8 CDCLVC1104PW, IC9 TPD4E001QDBVRQ1, J1 2.54-2*5, J2 2.54-2*5, J3 PM2.54-2*10, J6 2.54-2*5, J7 Conn_02x02_Counter_Clockwise, J8 Conn_02x02_Counter_Clockwise, J9 Conn_02x07_Odd_Even, M1 Conn_01x01_Socket, M2 Conn_01x01_Socket, M3 Conn_01x01_Socket, M4 Conn_01x01_Socket, M5 Conn_01x01_Socket, M6 Conn_01x01_Socket, M7 Conn_01x01_Socket, M8 Conn_01x01_Socket, Q1 FMMT618TA, Q10 TPT1042VQ-SO1R-S, Q11 AT24C16C-SSHM-T, Q12 SN74LVC14APWRG4, Q2 FMMT618TA, Q3 CP2102N-A02-GQFN28R, Q4 FMMT618TA, Q5 AMS1117-3.3, Q50 SN74LVC14APWRG4, Q6 TYPEC-304-ACP16, Q7 FMMT618TA, Q8 SRV05-4HTG, Q9 TPT1042VQ-SO1R-S, SW1 SW_DIP_x02, SW2 SW_Push, U1 ADR423ARMZ, X1 20MHz, X2 20MHz, Y1 ECS-2520S33-250-FN-TR

Commit message: 增加16Pins ADC接口，修改EtherCAT接口顺序，修改ADR423输入电源电压为5V
Parts:
- added J4: Conn_01x16_Pin, 1mmlab_footprint:CONN-TH_250-216, symbol Connector:Conn_01x16_Pin
- added R345: 10k, Resistor_SMD:R_0402_1005Metric, symbol Device:R_Small
- added R350, R351, R352, R353, R354, R355, R356, R357, R358, R359, R360, R361, R362, R363, R364, R365: DNP, Resistor_SMD:R_0603_1608Metric, symbol Device:R
Connections:
- net +3V3A_DSP: no longer C40.1, C43.1, U1.2 (VIN)
- net ADC_14: now also R364.2
- net ADC_15: now also R365.2
- net ADC_A4: now also R351.2
- net ADC_A5: now also R350.2
- net ADC_B4: now also R352.2
- net ADC_B5: now also R353.2
- net ADC_C2: now also R360.2
- net ADC_C3: now also R361.2
- net ADC_C4: now also R362.2
- net ADC_C5: now also R363.2
- net ADC_D0: now also R354.2
- net ADC_D1: now also R359.2
- net ADC_D2: now also R355.2
- net ADC_D3: now also R356.2
- net ADC_D4: now also R357.2
- net ADC_D5: now also R358.2
- net D+5V: now also C40.1, C43.1, U1.2 (VIN)
- net GND: now also R345.1
- net ERRORSTS: now reaches IC1.U19 (ERRORSTS)
- net ERRORSTS: now also R345.2
- new net: J4.8 (Pin_8), R356.1
- new net: J4.1 (Pin_1), R350.1
- new net: J4.10 (Pin_10), R358.1
- new net: J4.11 (Pin_11), R360.1
- new net: J4.12 (Pin_12), R361.1
- new net: J4.13 (Pin_13), R362.1
- new net: J4.14 (Pin_14), R363.1
- new net: J4.15 (Pin_15), R364.1
- new net: J4.16 (Pin_16), R365.1
- new net: J4.2 (Pin_2), R351.1
- new net: J4.3 (Pin_3), R352.1
- new net: J4.4 (Pin_4), R353.1
- new net: J4.5 (Pin_5), R354.1
- new net: J4.6 (Pin_6), R359.1
- new net: J4.7 (Pin_7), R355.1
- new net: J4.9 (Pin_9), R357.1

Commit message: 修复AGND BUG
Connections:
- net AGND is gone; now on net GND: C10.2, C11.1, C12.2, C13.1, C14.2, C15.2, C16.1, C17.2, C18.2, C19.1, C20.1, C21.1, C214.2, C22.2, C23.1, C24.2, C25.1, C26.1, C27.2, CN1.2, CN1.4, CN2.2, CN2.4, D12.3, D13.3, D14.1 (A), D15.1 (A), DSUB1.9, DSUB2.9, DSUB3.9, DSUB4.9, DSUB5.8, DSUB5.9, DSUB6.8, DSUB6.9, J6.1, J6.2, J6.3, J6.4, J6.5, J6.6, J7.2 (Pin_2), J8.2 (Pin_2), Q10.2 (GND), Q12.7 (GND), Q50.7 (GND), Q9.2 (GND), R31.1, R32.1, R45.2, R46.2, X1.2 (Gnd), X2.2 (Gnd)
