File: 28388BGA/ETHERCAT2.kicad_sch (KiCad schematic)
At the start: 37 parts, among them Q14 DP83822IRHBR

Commit message: 增加16Pins ADC接口，修改EtherCAT接口顺序，修改ADR423输入电源电压为5V
Parts:
- removed RJ1.1: HR871210DE, Lib4:RJ45-TH_HR871210DE, symbol sheet1-altium-import:HR871210DE
- added RJ1.1: HR871210DE, Lib4:RJ45-TH_HR871210DE, symbol sheet1-altium-import:HR871210DE
Connections:
- net +3V3D_DSP: now also RJ1.1.P3 (RCT), RJ1.1.P4 (TCT)
- net ESC_LED_LINK: now also RJ1.1.P10 (10)
- net ESC_PHY: now also RJ1.1.P12 (12)
- net GND: now also RJ1.1.P8 (CHS_GND)
- net at Q14.12 (TD_P), R100.1: now also RJ1.1.P5 (TD+)
- net at Q14.10 (RD_P), R103.1: now also RJ1.1.P1 (RD+)
- net at R106.2: now also RJ1.1.P11 (11)
- net at Q14.9 (RD_M), R104.1: now also RJ1.1.P2 (RD-)
- net at Q14.11 (TD_M), R101.1: now also RJ1.1.P6 (TD-)
- net at R105.2: now also RJ1.1.P9 (9)
Changed lines of the file:
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@@
 	)
 	(junction
-		(at 292.1 128.27)
-		(diameter 0)
-		(color 0 0 0 0)
-	)
-	(junction
 		(at 85.09 50.8)
 		(diameter 0)
@@
 	(wire
 		(pts
-			(xy 287.02 123.19) (xy 292.1 123.19)
-		)
-		(stroke
-			(width 0)
-			(type default)
-		)
-	)
-	(wire
-		(pts
 			(xy 135.89 104.14) (xy 143.51 104.14)
 		)
@@
 	(wire
 		(pts
-			(xy 292.1 128.27) (xy 292.1 129.54)
-		)
-		(stroke
-			(width 0)
-			(type default)
-		)
-	)
-	(wire
-		(pts
 			(xy 171.45 45.72) (xy 168.91 45.72)
 		)
@@
 	(wire
 		(pts
-			(xy 287.02 128.27) (xy 292.1 128.27)
-		)
-		(stroke
-			(width 0)
-			(type default)
-		)
-	)
-	(wire
-		(pts
 			(xy 77.47 116.84) (xy 34.29 116.84)
 		)
@@
 	(wire
 		(pts
-			(xy 292.1 123.19) (xy 292.1 128.27)
-		)
-		(stroke
-			(width 0)
-			(type default)
-		)
-	)
-	(wire
-		(pts
 			(xy 189.23 44.45) (xy 181.61 44.45)
 		)
@@
 	)
 	(symbol
-		(lib_id "sheet1-altium-import:HR871210DE")
-		(at 259.08 107.95 0)
-		(unit 1)
-		(exclude_from_sim no)
-		(in_bom yes)
-		(on_board yes)
-		(dnp no)
-		(fields_autoplaced yes)
-		(property "Reference" "RJ1.1"
-			(at 259.08 78.74 0)
-			(effects
-				(font
-					(face "Arial")
-					(size 1.6891 1.6891)
-				)
-			)
-		)
-		(property "Value" "HR871210DE"
-			(at 259.08 82.55 0)
-			(effects
-				(font
-					(face "Arial")
-					(size 1.6891 1.6891)
-				)
-			)
-		)
-		(property "Footprint" "Lib4:RJ45-TH_HR871210DE"
-			(at 259.08 107.95 0)
-			(effects
-				(font
-					(size 1.27 1.27)
-				)
-				(hide yes)
-			)
-		)
-		(property "Datasheet" ""
-			(at 259.08 107.95 0)
-			(effects
-				(font
-					(size 1.27 1.27)
-				)
-				(hide yes)
-			)
-		)
-		(property "Description" ""
-			(at 259.08 107.95 0)
-			(effects
-				(font
-					(size 1.27 1.27)
-				)
-				(hide yes)
-			)
-		)
-		(property "Manufacturer Part" "HR871210DE"
-			(at 259.08 107.95 0)
-			(effects
-				(font
-					(size 1.27 1.27)
-				)
-				(hide yes)
-			)
-		)
-		(property "Manufacturer" "HANRUN(汉仁)"
-			(at 259.08 107.95 0)
-			(effects
-				(font
-					(size 1.27 1.27)
-				)
-				(hide yes)
-			)
-		)
-		(property "Supplier Part" "C19724758"
-			(at 259.08 107.95 0)
-			(effects
-				(font
-					(size 1.27 1.27)
-				)
-				(hide yes)
-			)
-		)
-		(property "Supplier" "LCSC"
-			(at 259.08 107.95 0)
-			(effects
-				(font
-					(size 1.27 1.27)
-				)
-				(hide yes)
-			)
-		)
-		(pin "7"
-		)
-		(pin "4"
-		)
-		(pin "5"
-		)
-		(pin "1"
-		)
-		(pin "9"
-		)
-		(pin "10"
-		)
-		(pin "12"
-		)
-		(pin "6"
-		)
-		(pin "3"
-		)
-		(pin "11"
-		)
-		(pin "2"
-		)
-		(pin "8"
-		)
-		(pin "13"
-		)
-		(pin "14"
-		)
-		(pin "P2"
-		)
-		(pin "P6"
-		)
-		(pin "P1"
-		)
-		(pin "P4"
-		)
-		(pin "P7"
-		)
-		(pin "P8"
-		)
-		(pin "P9"
-		)
-		(pin "P3"
-		)
-		(pin "P5"
-		)
-		(pin "P12"
-		)
-		(pin "P11"
-		)
-		(pin "P10"
-		)
-		(instances
-			(project "28388bga"
-				(path "/88c87a56-bf0e-49aa-812f-d0846700c8ff/17fd3f57-3bad-4b3f-9846-9b737a2222f4"
-					(reference "RJ1.1")
-					(unit 1)
-				)
-			)
-		)
-	)
-	(symbol
 		(lib_id "power:+3V3")
 		(at 246.38 52.07 0)
@@
 	)
 	(symbol
-		(lib_id "power:Earth_Protective")
-		(at 292.1 128.27 90)
-		(unit 1)
-		(exclude_from_sim no)
-		(in_bom yes)
-		(on_board yes)
-		(dnp no)
-		(property "Reference" "#PWR0263"
-			(at 292.1 128.27 0)
-			(effects
-				(font
-					(size 1.27 1.27)
-				)
-				(hide yes)
-			)
-		)
-		(property "Value" "PE_GND"
-			(at 298.45 128.27 0)
-			(effects
-				(font
-					(size 1.27 1.27)
-				)
-			)
-		)
-		(property "Footprint" ""
-			(at 294.64 128.27 0)
-			(effects
-				(font
-					(size 1.27 1.27)
-				)
-				(hide yes)
-			)
-		)
-		(property "Datasheet" "~"
-			(at 294.64 128.27 0)
-			(effects
-				(font
-					(size 1.27 1.27)
-				)
-				(hide yes)
-			)
-		)
-		(property "Description" "Power symbol creates a global label with name \"Earth_Protective\""
-			(at 292.1 128.27 0)
-			(effects
-				(font
-					(size 1.27 1.27)
-				)
-				(hide yes)
-			)
-		)
-		(pin "1"
-		)
-		(instances
-			(project "28388bga"
-				(path "/88c87a56-bf0e-49aa-812f-d0846700c8ff/17fd3f57-3bad-4b3f-9846-9b737a2222f4"
-					(reference "#PWR0263")
-					(unit 1)
-				)
-			)
-		)
-	)
-	(symbol
 		(lib_id "sheet1-altium-import:CAP_2")
 		(at 81.28 48.26 180)
@@
 				)
 			)
+		)
+	)
+	(symbol
+		(lib_id "sheet1-altium-import:HR871210DE")
+		(at 259.08 107.95 0)
+		(unit 2)
+		(exclude_from_sim no)
+		(in_bom yes)
+		(on_board yes)
+		(dnp no)
+		(fields_autoplaced yes)
+		(property "Reference" "RJ1.1"
+			(at 283.21 106.0449 0)
+			(effects
+				(font
+					(face "Arial")
+					(size 1.6891 1.6891)
+				)
+				(justify left)
+			)
+		)
+		(property "Value" "HR871210DE"
+			(at 283.21 109.8549 0)
+			(effects
+				(font
+					(face "Arial")
+					(size 1.6891 1.6891)
+				)
+				(justify left)
+			)
+		)
+		(property "Footprint" "Lib4:RJ45-TH_HR871210DE"
+			(at 259.08 107.95 0)
+			(effects
+				(font
+					(size 1.27 1.27)
+				)
+				(hide yes)
+			)
+		)
+		(property "Datasheet" ""
+			(at 259.08 107.95 0)
+			(effects
+				(font
+					(size 1.27 1.27)
+				)
+				(hide yes)
+			)
+		)
+		(property "Description" ""
+			(at 259.08 107.95 0)
+			(effects
+				(font
+					(size 1.27 1.27)
+				)
+				(hide yes)
+			)
+		)
+		(property "Manufacturer Part" "HR871210DE"
+			(at 259.08 107.95 0)
+			(effects
+				(font
+					(size 1.27 1.27)
+				)
+				(hide yes)
+			)
+		)
+		(property "Manufacturer" "HANRUN(汉仁)"
+			(at 259.08 107.95 0)
+			(effects
+				(font
+					(size 1.27 1.27)
+				)
+				(hide yes)
+			)
+		)
+		(property "Supplier Part" "C19724758"
+			(at 259.08 107.95 0)
+			(effects
+				(font
+					(size 1.27 1.27)
+				)
+				(hide yes)
+			)
+		)
+		(property "Supplier" "LCSC"
+			(at 259.08 107.95 0)
+			(effects
+				(font
+					(size 1.27 1.27)
+				)
+				(hide yes)
+			)
+		)
+		(pin "7"
+		)
+		(pin "4"
+		)
+		(pin "5"
+		)
+		(pin "1"
+		)
+		(pin "9"
+		)
+		(pin "10"
+		)
+		(pin "12"
+		)
+		(pin "6"
+		)
+		(pin "3"
+		)
+		(pin "11"
+		)
+		(pin "2"
+		)
+		(pin "8"
+		)
+		(pin "13"
+		)
+		(pin "14"
+		)
+		(pin "P2"
+		)
+		(pin "P6"
+		)
+		(pin "P1"
+		)
+		(pin "P4"
+		)
+		(pin "P7"
+		)
+		(pin "P8"
+		)
+		(pin "P9"
+		)
+		(pin "P3"
+		)
+		(pin "P5"
+		)
+		(pin "P12"
+		)
+		(pin "P11"
+		)
+		(pin "P10"
+		)
+		(instances
+			(project "28388bga"
+				(path "/88c87a56-bf0e-49aa-812f-d0846700c8ff/17fd3f57-3bad-4b3f-9846-9b737a2222f4"
+					(reference "RJ1.1")
+					(unit 2)
+				)
+			)
