File: 28388BGA/H485.kicad_sch (KiCad schematic)
At the start: 22 parts, among them CN7 DB141V-2.54-6P, Q43 TPT75176B-SO1R, Q44 SN74LVC1G125DCKR

Commit message: 修复AGND BUG
Connections:
- net AGND renamed GND
Changed lines of the file:
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@@
 		(on_board yes)
 		(dnp no)
-		(property "Reference" "#PWR0445"
-			(at 135.89 104.14 0)
+		(property "Reference" "#PWR445"
+			(at 135.89 110.49 0)
 			(effects
 				(font
@@
 			)
 		)
-		(property "Value" "AGND"
-			(at 138.43 110.744 0)
+		(property "Value" "GND"
+			(at 135.89 107.95 0)
 			(effects
 				(font
 					(size 1.27 1.27)
 				)
-				(justify right)
-				(hide yes)
 			)
 		)
@@
 			(project "28388bga"
 				(path "/88c87a56-bf0e-49aa-812f-d0846700c8ff/b1d8f62e-8e7d-4d1c-ae44-e51a79ec0caa"
-					(reference "#PWR0445")
+					(reference "#PWR445")
 					(unit 1)
 				)
 				(path "/88c87a56-bf0e-49aa-812f-d0846700c8ff/e5b9647e-3d6c-4de7-89bf-da21707104e7"
-					(reference "#PWR0461")
+					(reference "#PWR461")
 					(unit 1)
 				)
@@
 		(on_board yes)
 		(dnp no)
-		(property "Reference" "#PWR0442"
-			(at 97.79 118.11 0)
+		(property "Reference" "#PWR442"
+			(at 97.79 124.46 0)
 			(effects
 				(font
@@
 			)
 		)
-		(property "Value" "AGND"
-			(at 97.79 125.984 0)
+		(property "Value" "GND"
+			(at 97.79 121.92 0)
 			(effects
 				(font
 					(size 1.27 1.27)
 				)
-				(hide yes)
 			)
 		)
@@
 			(project "28388bga"
 				(path "/88c87a56-bf0e-49aa-812f-d0846700c8ff/b1d8f62e-8e7d-4d1c-ae44-e51a79ec0caa"
-					(reference "#PWR0442")
+					(reference "#PWR442")
 					(unit 1)
 				)
 				(path "/88c87a56-bf0e-49aa-812f-d0846700c8ff/e5b9647e-3d6c-4de7-89bf-da21707104e7"
-					(reference "#PWR0458")
+					(reference "#PWR458")
 					(unit 1)
 				)
@@
 		(on_board yes)
 		(dnp no)
-		(property "Reference" "#PWR0444"
-			(at 130.81 76.2 0)
+		(property "Reference" "#PWR444"
+			(at 130.81 82.55 0)
 			(effects
 				(font
@@
 			)
 		)
-		(property "Value" "AGND"
-			(at 133.35 82.804 0)
+		(property "Value" "GND"
+			(at 130.81 80.01 0)
 			(effects
 				(font
 					(size 1.27 1.27)
 				)
-				(justify right)
-				(hide yes)
 			)
 		)
@@
 			(project "28388bga"
 				(path "/88c87a56-bf0e-49aa-812f-d0846700c8ff/b1d8f62e-8e7d-4d1c-ae44-e51a79ec0caa"
-					(reference "#PWR0444")
+					(reference "#PWR444")
 					(unit 1)
 				)
 				(path "/88c87a56-bf0e-49aa-812f-d0846700c8ff/e5b9647e-3d6c-4de7-89bf-da21707104e7"
-					(reference "#PWR0460")
+					(reference "#PWR460")
 					(unit 1)
 				)
@@
 		(on_board yes)
 		(dnp no)
-		(property "Reference" "#PWR0443"
-			(at 100.33 66.04 0)
+		(property "Reference" "#PWR443"
+			(at 100.33 72.39 0)
 			(effects
 				(font
@@
 			)
 		)
-		(property "Value" "AGND"
-			(at 102.87 72.644 0)
+		(property "Value" "GND"
+			(at 100.33 69.85 0)
 			(effects
 				(font
 					(size 1.27 1.27)
 				)
-				(justify right)
-				(hide yes)
 			)
 		)
@@
 			(project "28388bga"
 				(path "/88c87a56-bf0e-49aa-812f-d0846700c8ff/b1d8f62e-8e7d-4d1c-ae44-e51a79ec0caa"
-					(reference "#PWR0443")
+					(reference "#PWR443")
 					(unit 1)
 				)
 				(path "/88c87a56-bf0e-49aa-812f-d0846700c8ff/e5b9647e-3d6c-4de7-89bf-da21707104e7"
-					(reference "#PWR0459")
+					(reference "#PWR459")
 					(unit 1)
 				)
@@
 		(on_board yes)
 		(dnp no)
-		(property "Reference" "#PWR0454"
-			(at 218.44 104.14 0)
+		(property "Reference" "#PWR454"
+			(at 218.44 110.49 0)
 			(effects
 				(font
@@
 			)
 		)
-		(property "Value" "AGND"
-			(at 220.98 110.744 0)
+		(property "Value" "GND"
+			(at 218.44 107.95 0)
 			(effects
 				(font
 					(size 1.27 1.27)
 				)
-				(justify right)
-				(hide yes)
 			)
 		)
@@
 			(project "28388bga"
 				(path "/88c87a56-bf0e-49aa-812f-d0846700c8ff/b1d8f62e-8e7d-4d1c-ae44-e51a79ec0caa"
-					(reference "#PWR0454")
+					(reference "#PWR454")
 					(unit 1)
 				)
 				(path "/88c87a56-bf0e-49aa-812f-d0846700c8ff/e5b9647e-3d6c-4de7-89bf-da21707104e7"
-					(reference "#PWR0470")
+					(reference "#PWR470")
 					(unit 1)
 				)
@@
 		(on_board yes)
 		(dnp no)
-		(property "Reference" "#PWR0448"
-			(at 148.59 111.76 0)
+		(property "Reference" "#PWR448"
+			(at 148.59 118.11 0)
 			(effects
 				(font
@@
 			)
 		)
-		(property "Value" "AGND"
-			(at 151.13 118.364 0)
+		(property "Value" "GND"
+			(at 148.59 115.57 0)
 			(effects
 				(font
 					(size 1.27 1.27)
 				)
-				(justify right)
-				(hide yes)
 			)
 		)
@@
 			(project "28388bga"
 				(path "/88c87a56-bf0e-49aa-812f-d0846700c8ff/b1d8f62e-8e7d-4d1c-ae44-e51a79ec0caa"
-					(reference "#PWR0448")
+					(reference "#PWR448")
 					(unit 1)
 				)
 				(path "/88c87a56-bf0e-49aa-812f-d0846700c8ff/e5b9647e-3d6c-4de7-89bf-da21707104e7"
-					(reference "#PWR0464")
+					(reference "#PWR464")
 					(unit 1)
 				)
@@
 		(on_board yes)
 		(dnp no)
-		(property "Reference" "#PWR0453"
-			(at 205.74 91.44 0)
+		(property "Reference" "#PWR453"
+			(at 212.09 91.44 0)
 			(effects
 				(font
@@
 			)
 		)
-		(property "Value" "AGND"
-			(at 212.344 88.9 0)
+		(property "Value" "GND"
+			(at 209.55 91.44 0)
 			(effects
 				(font
 					(size 1.27 1.27)
 				)
-				(justify right)
-				(hide yes)
 			)
 		)
@@
 			(project "28388bga"
 				(path "/88c87a56-bf0e-49aa-812f-d0846700c8ff/b1d8f62e-8e7d-4d1c-ae44-e51a79ec0caa"
-					(reference "#PWR0453")
+					(reference "#PWR453")
 					(unit 1)
 				)
 				(path "/88c87a56-bf0e-49aa-812f-d0846700c8ff/e5b9647e-3d6c-4de7-89bf-da21707104e7"
-					(reference "#PWR0469")
+					(reference "#PWR469")
 					(unit 1)
 				)
@@
 		(on_board yes)
 		(dnp no)
-		(property "Reference" "#PWR0451"
-			(at 166.37 111.76 0)
+		(property "Reference" "#PWR451"
+			(at 166.37 118.11 0)
 			(effects
 				(font
@@
 			)
 		)
-		(property "Value" "AGND"
-			(at 168.91 118.364 0)
+		(property "Value" "GND"
+			(at 166.37 115.57 0)
 			(effects
 				(font
 					(size 1.27 1.27)
 				)
-				(justify right)
-				(hide yes)
 			)
 		)
@@
 			(project "28388bga"
 				(path "/88c87a56-bf0e-49aa-812f-d0846700c8ff/b1d8f62e-8e7d-4d1c-ae44-e51a79ec0caa"
-					(reference "#PWR0451")
+					(reference "#PWR451")
 					(unit 1)
 				)
 				(path "/88c87a56-bf0e-49aa-812f-d0846700c8ff/e5b9647e-3d6c-4de7-89bf-da21707104e7"
-					(reference "#PWR0467")
+					(reference "#PWR467")
 					(unit 1)
 				)
@@
 		(on_board yes)
 		(dnp no)
-		(property "Reference" "#PWR0450"
-			(at 160.02 48.26 0)
+		(property "Reference" "#PWR450"
+			(at 160.02 54.61 0)
 			(effects
 				(font
@@
 			)
 		)
-		(property "Value" "AGND"
-			(at 162.56 54.864 0)
+		(property "Value" "GND"
+			(at 160.02 52.07 0)
 			(effects
 				(font
 					(size 1.27 1.27)
 				)
-				(justify right)
-				(hide yes)
 			)
 		)
@@
 			(project "28388bga"
 				(path "/88c87a56-bf0e-49aa-812f-d0846700c8ff/b1d8f62e-8e7d-4d1c-ae44-e51a79ec0caa"
-					(reference "#PWR0450")
+					(reference "#PWR450")
 					(unit 1)
 				)
 				(path "/88c87a56-bf0e-49aa-812f-d0846700c8ff/e5b9647e-3d6c-4de7-89bf-da21707104e7"
-					(reference "#PWR0466")
+					(reference "#PWR466")
 					(unit 1)
 				)
@@
 		(on_board yes)
 		(dnp no)
-		(property "Reference" "#PWR0452"
-			(at 176.53 111.76 0)
+		(property "Reference" "#PWR452"
+			(at 176.53 118.11 0)
 			(effects
 				(font
@@
 			)
 		)
-		(property "Value" "AGND"
-			(at 179.07 118.364 0)
+		(property "Value" "GND"
+			(at 176.53 115.57 0)
 			(effects
 				(font
 					(size 1.27 1.27)
 				)
-				(justify right)
-				(hide yes)
 			)
 		)
@@
 			(project "28388bga"
 				(path "/88c87a56-bf0e-49aa-812f-d0846700c8ff/b1d8f62e-8e7d-4d1c-ae44-e51a79ec0caa"
-					(reference "#PWR0452")
+					(reference "#PWR452")
 					(unit 1)
 				)
 				(path "/88c87a56-bf0e-49aa-812f-d0846700c8ff/e5b9647e-3d6c-4de7-89bf-da21707104e7"
-					(reference "#PWR0468")
+					(reference "#PWR468")
 					(unit 1)
 				)
