File: 28388core/ETHERCAT.kicad_sch (KiCad schematic)
At the start: 37 parts, among them Q13 DP83822IRHBR

Commit message: 1. usb 稳压、防倒灌 1 2. 仿真器贴片 1 3. EtherCAT确认 1 4. EtherCAT差分信号 5. 金手指选型换1.6 要不就1.0？
Connections:
- net RD_P: now reaches Q13.10 (RD_P), R84.1, RJ1.1.1 (RD+)
- net RD_M: now reaches Q13.9 (RD_M), R85.1, RJ1.1.2 (RD-)
- net TD_P: now reaches Q13.12 (TD_P), R81.1, RJ1.1.5 (TD+)
- net TD_M: now reaches Q13.11 (TD_M), R82.1, RJ1.1.6 (TD-)
Changed lines of the file:
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@@
+	)
+	(junction
+		(at 166.37 71.12)
+		(diameter 0)
+		(color 0 0 0 0)
+	)
+	(junction
+		(at 171.45 68.58)
+		(diameter 0)
+		(color 0 0 0 0)
 	)
 	(junction
@@
 	)
 	(junction
+		(at 140.97 76.2)
+		(diameter 0)
+		(color 0 0 0 0)
+	)
+	(junction
 		(at 165.1 99.06)
 		(diameter 0)
@@
 	(junction
 		(at 46.99 82.55)
+		(diameter 0)
+		(color 0 0 0 0)
+	)
+	(junction
+		(at 135.89 78.74)
 		(diameter 0)
 		(color 0 0 0 0)
@@
 	(wire
 		(pts
+			(xy 171.45 68.58) (xy 149.86 68.58)
+		)
+		(stroke
+			(width 0)
+			(type default)
+		)
+	)
+	(wire
+		(pts
 			(xy 76.2 81.28) (xy 69.85 81.28)
 		)
@@
 	(wire
 		(pts
-			(xy 196.85 71.12) (xy 154.94 71.12)
+			(xy 196.85 71.12) (xy 166.37 71.12)
 		)
 		(stroke
@@
 	(wire
 		(pts
+			(xy 171.45 58.42) (xy 171.45 68.58)
+		)
+		(stroke
+			(width 0)
+			(type default)
+		)
+	)
+	(wire
+		(pts
 			(xy 134.62 101.6) (xy 142.24 101.6)
 		)
@@
 	(wire
 		(pts
+			(xy 135.89 78.74) (xy 172.72 78.74)
+		)
+		(stroke
+			(width 0)
+			(type default)
+		)
+	)
+	(wire
+		(pts
 			(xy 36.83 48.26) (xy 45.72 48.26)
 		)
@@
 	(wire
 		(pts
-			(xy 134.62 78.74) (xy 172.72 78.74)
+			(xy 134.62 78.74) (xy 135.89 78.74)
 		)
 		(stroke
@@
 	(wire
 		(pts
+			(xy 166.37 71.12) (xy 154.94 71.12)
+		)
+		(stroke
+			(width 0)
+			(type default)
+		)
+	)
+	(wire
+		(pts
 			(xy 55.88 73.66) (xy 55.88 38.1)
 		)
@@
 	(wire
 		(pts
+			(xy 135.89 55.88) (xy 135.89 78.74)
+		)
+		(stroke
+			(width 0)
+			(type default)
+		)
+	)
+	(wire
+		(pts
 			(xy 52.07 82.55) (xy 46.99 82.55)
 		)
@@
 	(wire
 		(pts
+			(xy 140.97 53.34) (xy 140.97 76.2)
+		)
+		(stroke
+			(width 0)
+			(type default)
+		)
+	)
+	(wire
+		(pts
 			(xy 17.78 104.14) (xy 15.24 104.14)
 		)
@@
 	(wire
 		(pts
+			(xy 140.97 76.2) (xy 165.1 76.2)
+		)
+		(stroke
+			(width 0)
+			(type default)
+		)
+	)
+	(wire
+		(pts
 			(xy 154.94 43.18) (xy 157.48 43.18)
 		)
@@
 	(wire
 		(pts
-			(xy 203.2 68.58) (xy 149.86 68.58)
+			(xy 203.2 68.58) (xy 171.45 68.58)
 		)
 		(stroke
@@
 	(wire
 		(pts
-			(xy 134.62 76.2) (xy 165.1 76.2)
+			(xy 134.62 76.2) (xy 140.97 76.2)
+		)
+		(stroke
+			(width 0)
+			(type default)
+		)
+	)
+	(wire
+		(pts
+			(xy 166.37 60.96) (xy 166.37 71.12)
 		)
 		(stroke
@@
 			(width 0)
 			(type default)
+		)
+	)
+	(hierarchical_label "TD_P"
+		(shape output)
+		(at 171.45 58.42 90)
+		(effects
+			(font
+				(size 1.27 1.27)
+			)
+			(justify left)
 		)
 	)
@@
 		)
 	)
+	(hierarchical_label "RD_M"
+		(shape output)
+		(at 135.89 55.88 90)
+		(effects
+			(font
+				(size 1.27 1.27)
+			)
+			(justify left)
+		)
+	)
+	(hierarchical_label "RD_P"
+		(shape output)
+		(at 140.97 53.34 90)
+		(effects
+			(font
+				(size 1.27 1.27)
+			)
+			(justify left)
+		)
+	)
 	(hierarchical_label "ESC_TX_D3"
 		(shape input)
@@
 		)
 	)
+	(hierarchical_label "TD_M"
+		(shape output)
+		(at 166.37 60.96 90)
+		(effects
+			(font
+				(size 1.27 1.27)
+			)
+			(justify left)
+		)
+	)
