File: 28388core/ETHERCAT2.kicad_sch (KiCad schematic)
At the start: 37 parts, among them Q14 DP83822IRHBR

Commit message: 1. usb 稳压、防倒灌 1 2. 仿真器贴片 1 3. EtherCAT确认 1 4. EtherCAT差分信号 5. 金手指选型换1.6 要不就1.0？
Connections:
- net TD_P: now reaches Q14.12 (TD_P), R100.1, RJ1.1.P5 (TD+)
- net RD_M: now reaches Q14.9 (RD_M), R104.1, RJ1.1.P2 (RD-)
- net RD_P: now reaches Q14.10 (RD_P), R103.1, RJ1.1.P1 (RD+)
- net TD_M: now reaches Q14.11 (TD_M), R101.1, RJ1.1.P6 (TD-)
Changed lines of the file:
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@@
+	)
+	(junction
+		(at 167.64 73.66)
+		(diameter 0)
+		(color 0 0 0 0)
 	)
 	(junction
@@
 	)
 	(junction
+		(at 137.16 81.28)
+		(diameter 0)
+		(color 0 0 0 0)
+	)
+	(junction
 		(at 167.64 137.16)
 		(diameter 0)
@@
 	)
 	(junction
+		(at 142.24 78.74)
+		(diameter 0)
+		(color 0 0 0 0)
+	)
+	(junction
 		(at 85.09 50.8)
 		(diameter 0)
@@
 	(junction
 		(at 29.21 114.3)
+		(diameter 0)
+		(color 0 0 0 0)
+	)
+	(junction
+		(at 172.72 71.12)
 		(diameter 0)
 		(color 0 0 0 0)
@@
 	(wire
 		(pts
-			(xy 201.93 71.12) (xy 151.13 71.12)
-		)
-		(stroke
-			(width 0)
-			(type default)
-		)
-	)
-	(wire
-		(pts
 			(xy 135.89 104.14) (xy 143.51 104.14)
 		)
@@
 	(wire
 		(pts
-			(xy 135.89 81.28) (xy 173.99 81.28)
+			(xy 135.89 81.28) (xy 137.16 81.28)
 		)
 		(stroke
@@
 	(wire
 		(pts
+			(xy 137.16 81.28) (xy 173.99 81.28)
+		)
+		(stroke
+			(width 0)
+			(type default)
+		)
+	)
+	(wire
+		(pts
 			(xy 16.51 111.76) (xy 24.13 111.76)
 		)
@@
 	(wire
 		(pts
+			(xy 137.16 58.42) (xy 137.16 81.28)
+		)
+		(stroke
+			(width 0)
+			(type default)
+		)
+	)
+	(wire
+		(pts
 			(xy 138.43 134.62) (xy 135.89 134.62)
 		)
@@
 	(wire
 		(pts
+			(xy 142.24 78.74) (xy 166.37 78.74)
+		)
+		(stroke
+			(width 0)
+			(type default)
+		)
+	)
+	(wire
+		(pts
 			(xy 78.74 40.64) (xy 85.09 40.64)
 		)
@@
 	(wire
 		(pts
+			(xy 167.64 73.66) (xy 156.21 73.66)
+		)
+		(stroke
+			(width 0)
+			(type default)
+		)
+	)
+	(wire
+		(pts
 			(xy 135.89 71.12) (xy 151.13 71.12)
 		)
@@
 	(wire
 		(pts
+			(xy 172.72 71.12) (xy 151.13 71.12)
+		)
+		(stroke
+			(width 0)
+			(type default)
+		)
+	)
+	(wire
+		(pts
 			(xy 53.34 104.14) (xy 77.47 104.14)
 		)
@@
 	(wire
 		(pts
+			(xy 172.72 60.96) (xy 172.72 71.12)
+		)
+		(stroke
+			(width 0)
+			(type default)
+		)
+	)
+	(wire
+		(pts
 			(xy 24.13 40.64) (xy 24.13 38.1)
 		)
@@
 	(wire
 		(pts
-			(xy 196.85 73.66) (xy 156.21 73.66)
+			(xy 196.85 73.66) (xy 167.64 73.66)
 		)
 		(stroke
@@
 	(wire
 		(pts
+			(xy 172.72 71.12) (xy 201.93 71.12)
+		)
+		(stroke
+			(width 0)
+			(type default)
+		)
+	)
+	(wire
+		(pts
 			(xy 156.21 100.33) (xy 156.21 99.06)
 		)
@@
 	(wire
 		(pts
-			(xy 135.89 78.74) (xy 166.37 78.74)
+			(xy 135.89 78.74) (xy 142.24 78.74)
 		)
 		(stroke
@@
 	(wire
 		(pts
+			(xy 142.24 55.88) (xy 142.24 78.74)
+		)
+		(stroke
+			(width 0)
+			(type default)
+		)
+	)
+	(wire
+		(pts
 			(xy 173.99 88.9) (xy 173.99 81.28)
 		)
@@
 		(pts
 			(xy 212.09 69.85) (xy 212.09 72.39)
+		)
+		(stroke
+			(width 0)
+			(type default)
+		)
+	)
+	(wire
+		(pts
+			(xy 167.64 63.5) (xy 167.64 73.66)
 		)
 		(stroke
@@
 		)
 	)
+	(hierarchical_label "RD_M"
+		(shape output)
+		(at 137.16 58.42 90)
+		(effects
+			(font
+				(size 1.27 1.27)
+			)
+			(justify left)
+		)
+	)
 	(hierarchical_label "ESC_RX_D3"
 		(shape input)
@@
 		)
 	)
+	(hierarchical_label "RD_P"
+		(shape output)
+		(at 142.24 55.88 90)
+		(effects
+			(font
+				(size 1.27 1.27)
+			)
+			(justify left)
+		)
+	)
 	(hierarchical_label "ESC_MDC"
 		(shape input)
@@
 		)
 	)
+	(hierarchical_label "TD_P"
+		(shape output)
+		(at 172.72 60.96 90)
+		(effects
+			(font
+				(size 1.27 1.27)
+			)
+			(justify left)
+		)
+	)
+	(hierarchical_label "TD_M"
+		(shape output)
+		(at 167.64 63.5 90)
+		(effects
+			(font
+				(size 1.27 1.27)
+			)
+			(justify left)
+		)
+	)
