File: 28388core/28388bga.kicad_pcb (KiCad board)
At the start: 8 copper layers, 70 x 100 mm, 309 parts, among them IC1 F28388DZWTS, IC2 TPS62420DRCT, IC6 OPA4350EA_250, IC7 TPS3702CX33DDCT, IC8 CDCLVC1104PW, IC9 TPS3702CX12DDCT, J9 Conn_02x07_Odd_Even, Q1 FMMT618TA, Q11 AT24C16C-SSHM-T, Q13 DP83822IRHBR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

Commit message: 修改电感封装
Parts:
- removed REF** (x6): Mark_TH_3mm, 1mmlab_footprint:Mark_TH_3mm
- removed REF** (x18): Mark_SMD, 1mmlab_footprint:Mark_SMD
- L4: footprint Inductor_SMD:L_Changjiang_FNR252012S -> Inductor_SMD:78438323032
- L5: footprint Inductor_SMD:L_Changjiang_FNR252012S -> Inductor_SMD:PFL3215
- moved C47 0.70 mm to (145.5, 131.3)
- moved FB2 0.62 mm to (148.3, 131.5)
- moved C56 0.44 mm to (151.2, 131.3)
- moved L5 0.22 mm to (143.0, 131.7)
Routing:
- net +3V3_DSP: track 43.7 -> 44.9 mm
