File: 28388motherboard/28388motherboard.kicad_sch (KiCad schematic)
At the start: 98 parts, among them CN10 DB141V-2.54-6P, CN9 DB141V-2.54-6P, J1 Conn_02x02_Counter_Clockwise, J11 2.54-2*5, J5 2.54-2*5, J6 2.54-2*5, J7 PM2.54-2*10, J8 Conn_02x02_Counter_Clockwise, Q47 AMS1117-3.3, Q48 TPT1042VQ-SO1R-S, Q49 TPT1042VQ-SO1R-S, Q50 FMMT618TA, Q51 FMMT618TA, Q52 FMMT618TA, Q53 FMMT618TA, X1 20MHz

Commit message: 底板分配引脚
Parts:
- added C121, C135: 0.1uF/50V, Capacitor_SMD:C_0603_1608Metric, symbol sheet1-altium-import:CAP_2
- added DSUB1: DDMRH15PFE006, Lib_sheet_10:DSUB-TH_15P-P2.29-H-F_DDMRH15PFE006, symbol sheet1-altium-import:DDMRH15PFE006
- added Q56: SN74LVC14APWRG4, Lib_sheet_10:TSSOP-14_L5.0-W4.4-P0.65-LS6.4-BL, symbol sheet1-altium-import:SN74LVC14APWRG4
- added X2: 20MHz, Lib_sheet_10:OSC-SMD_4P-L2.5-W2.0-BL, symbol sheet1-altium-import:ECS-2520S33-250-FN-TR
Connections:
- net GPIO0 is gone; now on net DSP-PWM1A: U3.12
- net GPIO1 is gone; now on net DSP-PWM1B: U3.14
- net GPIO10 is gone; now on net DSP-PWM6A: U2.47
- net GPIO11 is gone; now on net DSP-PWM6B: U2.43
- net GPIO123 is gone; now on net ADC_CLK_X1: U4.48
- net GPIO124 is gone; now on net ADC_DO_V_1: U4.45
- net GPIO126 is gone; now on net ADC_DO_W_1: U4.43
- net GPIO132 is gone; now on net ADC_DO_V_2: U4.15
- net GPIO134 is gone; now on net ADC_DO_W_2: U4.16
- net GPIO2 is gone; now on net DSP-PWM2A: U3.16
- net GPIO29 is gone; now on net DSP_A_CAN_EN: U4.37
- net GPIO3 is gone; now on net DSP-PWM2B: U3.19
- net GPIO30 is gone; now on net DSP_A_CAN_RX: U4.36
- net GPIO31 is gone; now on net DSP_A_CAN_TX: U4.38
- net GPIO37 is gone; now on net DSP_B_CAN_EN: U4.27
- net GPIO38 is gone; now on net DSP_B_CAN_TX: U4.23
- net GPIO39 is gone; now on net DSP_B_CAN_RX: U4.22
- net GPIO4 is gone; now on net DSP-PWM3A: U3.13
- net GPIO5 is gone; now on net DSP-PWM3B: U3.15
- net GPIO6 is gone; now on net DSP-PWM4A: U3.9
- net GPIO7 is gone; now on net DSP-PWM4B: U3.11
- net GPIO8 is gone; now on net DSP-PWM5A: U2.26
- net GPIO9 is gone; now on net DSP-PWM5B: U2.25
- net MSCLA is gone; now on net GPIO33: D41.3 (K), J5.5, J5.6
- net MSCLB is gone; now on net GPIO35: D43.3 (K), J11.5, J11.6
- net MSDAA is gone; now on net GPIO32: D42.3 (K), J5.7, J5.8
- net MSDAB is gone; now on net GPIO34: D44.3 (K), J11.7, J11.8
- net SPI_A_CK_HS is gone; now on net GPIO60: J7.2
- net SPI_A_MI_HS is gone; now on net GPIO59: J7.4
- net SPI_A_MO_HS is gone; now on net GPIO58: J7.1
- net SPI_B_CK_HS is gone; now on net GPIO27: SPI2.7 (Pin_7)
- net SPI_B_MO_HS is gone; now on net GPIO24: SPI2.1 (Pin_1)
- net SPI_C_CK_HS is gone; now on net GPIO102: SPI3.7 (Pin_7)
- net SPI_C_MI_HS is gone; now on net GPIO101: SPI3.2 (Pin_2)
- net SPI_C_MO_HS is gone; now on net GPIO100: SPI3.1 (Pin_1)
- net SPI_D_CK_HS is gone; now on net GPIO93: SPI4.7 (Pin_7)
- net SPI_D_MI_HS is gone; now on net GPIO92: SPI4.2 (Pin_2)
- net SPI_D_MO_HS is gone; now on net GPIO91: SPI4.1 (Pin_1)
- net ~{SPI_A_STE_HS} is gone; now on net GPIO61: J7.3
- net ~{SPI_B_STE_HS} is gone; now on net GPIO26: SPI2.8 (Pin_8)
- net ~{SPI_C_STE_HS} is gone; now on net GPIO103: SPI3.8 (Pin_8)
- net ~{SPI_D_STE_HS} is gone; now on net GPIO94: SPI4.8 (Pin_8)
- net D+5V: now also DSUB1.1
- net GND: now also C121.2, C135.2, DSUB1.8, DSUB1.9, Q56.7 (GND), X2.2 (Gnd)
- net PE_GND: now also DSUB1.16, DSUB1.17
- net VDD: now also C121.1, C135.1, Q56.14 (VCC), X2.4 (Vdd)
- net GPIO12 renamed DSP-PWM7A
- net GPIO122 renamed ADC_DO_U_1
- net GPIO13 renamed DSP-PWM7B
- net GPIO130 renamed ADC_DO_U_2
- net GPIO131 renamed ADC_CLK_X2
- net ADC_CLK_X2: now also X2.3 (Output)
- net GPIO14 renamed DSP-PWM8A
- net GPIO15 renamed DSP-PWM8B
- net GPIO16 renamed DSP-PWM9A
- net GPIO17 renamed DSP-PWM9B
- net GPIO18 renamed DSP-PWM10A
- net GPIO19 renamed DSP-PWM10B
- net GPIO20 renamed DSP-PWM11A
- net GPIO21 renamed DSP-PWM11B
- net GPIO22 renamed DSP-PWM12A
- net GPIO23 renamed DSP-PWM12B
- new net HALL_U: Q56.2 (1Y)
- new net HALL_UY: Q56.1 (1A)
- new net HALL_U_H: DSUB1.3
- new net HALL_U_L: DSUB1.2
- new net HALL_V: Q56.4 (2Y)
- new net HALL_VY: Q56.3 (2A)
- new net HALL_V_H: DSUB1.6
- new net HALL_V_L: DSUB1.7
- new net HALL_W: Q56.6 (3Y)
- new net HALL_WY: Q56.5 (3A)
- new net HALL_W_H: DSUB1.11
- new net HALL_W_L: DSUB1.12
- new net MQEP1A: Q56.12 (6Y)
- new net MQEP1AY: Q56.13 (6A)
- new net MQEP1A_H: DSUB1.15
- new net MQEP1A_L: DSUB1.10
- new net MQEP1B: Q56.10 (5Y)
- new net MQEP1BY: Q56.11 (5A)
- new net MQEP1B_H: DSUB1.5
- new net MQEP1B_L: DSUB1.4
- new net MQEP1Z: Q56.8 (4Y)
- new net MQEP1ZY: Q56.9 (4A)
- new net MQEP1Z_H: DSUB1.13
- new net MQEP1Z_L: DSUB1.14
- no-connect marks 13 -> 14
Other:
- added sheet 差分输入 (26c32.kicad_sch)
- added sheet 差分输入1 (26c32.kicad_sch)
- sheet IPM1 ports: added ADC_DO_U; removed none
- sheet IPM2 ports: added ADC_DO_U; removed none
- note added: "DELETE"
- note added: "HALL+EQEP=增量式编码器"
- moved on the sheet: C134, R287, R288, X1

Commit message: 完成第一版引脚分配
Parts:
- removed R291, R293: 1.69K/1%, Resistor_SMD:R_0805_2012Metric, symbol sheet1-altium-import:root_1_Res2
- removed R292, R294: 3.3K/1%, Resistor_SMD:R_0805_2012Metric, symbol sheet1-altium-import:root_1_Res2
- removed U2, U3, U4: ~, 1mmlab_footprint:CONN-SMD_50P-P0.50_XKB_X0515FVS-50CS-9TV01, symbol 1mmlab:X0515FVS-50AS-9TV01
- added C136: 0.1uF/50V, Capacitor_SMD:C_0603_1608Metric, symbol sheet1-altium-import:CAP_2
- added DSUB3: DDMRH15PFE006, Lib_sheet_10:DSUB-TH_15P-P2.29-H-F_DDMRH15PFE006, symbol sheet1-altium-import:DDMRH15PFE006
- added J10, J14: Conn_02x10_Top_Bottom, symbol Connector_Generic:Conn_02x10_Top_Bottom
- added J15, J16, J17, J18: Conn_02x02_Top_Bottom, symbol Connector_Generic:Conn_02x02_Top_Bottom
- added J3, J4, J9: ~, 1mmlab_footprint:CONN-SMD_50P-P0.50_XKB_X0515WVS-50AS-9TV01, symbol 1mmlab:X0515WVS-50AS-9TV01
- added Q57: SN74LVC14APWRG4, Lib_sheet_10:TSSOP-14_L5.0-W4.4-P0.65-LS6.4-BL, symbol sheet1-altium-import:SN74LVC14APWRG4
- added R291, R292: 10K, Resistor_SMD:R_0805_2012Metric, symbol sheet1-altium-import:root_2_Res2
Connections:
- net LED1 is gone; now on net GPIO115: R321.2
- net LED2 is gone; now on net GPIO116: R318.2
- net LED3 is gone; now on net GPIO117: R315.2
- net MQEP1AY is gone; now on net GPIO50: Q56.13 (6A)
- net MQEP1BY is gone; now on net GPIO51: Q56.11 (5A)
- net MQEP1ZY is gone; now on net GPIO53: Q56.9 (4A)
- net SPI_B_MI_HS is gone; now on net GPIO25: SPI2.2 (Pin_2)
- net 485_RTS_1: now also J9.7
- net 485_RTS_2: now also J4.24
- net ADC_A1_IN: now also J18.1 (Pin_1)
- net ADC_A2_IN: now also J18.2 (Pin_2)
- net ADC_A3_IN: now also J17.1 (Pin_1)
- net ADC_A4_IN: now also J17.2 (Pin_2)
- net ADC_CLK_X1: now also J10.11 (Pin_11), J9.42
- net ADC_CLK_X2: now also J14.11 (Pin_11), J9.34
- net ADC_DO_U_1: now also J16.4 (Pin_4)
- net ADC_DO_U_2: now also J15.4 (Pin_4)
- net ADC_DO_V_1: now also J9.40
- net ADC_DO_V_2: now also J9.43
- net ADC_DO_W_1: now also J9.38
- net ADC_DO_W_2: now also J9.22
- net D+5V: now also DSUB3.1, J10.1 (Pin_1), J10.2 (Pin_2), J14.1 (Pin_1), J14.2 (Pin_2), J3.18, J3.2, J3.34, J3.50, J4.18, J4.2, J4.34, J4.50, J9.2, J9.26, J9.50
- net DI-1-DSP-3.3V: now also J9.18, J9.21
- net DI-2-DSP-3.3V: now also J9.13, J9.28
- net DSP-PWM10A: now also J14.4 (Pin_4), J3.37
- net DSP-PWM10B: now also J14.7 (Pin_7), J3.39
- net DSP-PWM11A: now also J14.5 (Pin_5), J3.20
- net DSP-PWM11B: now also J14.8 (Pin_8), J3.31
- net DSP-PWM12A: now also J14.6 (Pin_6), J3.19
- net DSP-PWM12B: now also J14.9 (Pin_9), J3.11
- net DSP-PWM1A: now also J4.27
- net DSP-PWM1B: now also J4.15
- net DSP-PWM2A: now also J4.11
- net DSP-PWM2B: now also J4.8
- net DSP-PWM3A: now also J4.19
- net DSP-PWM3B: now also J4.7
- net DSP-PWM4A: now also J4.23
- net DSP-PWM4B: now also J4.6
- net DSP-PWM5A: now also J3.16
- net DSP-PWM5B: now also J3.27
- net DSP-PWM6A: now also J3.30
- net DSP-PWM6B: now also J3.38
- net DSP-PWM7A: now also J10.4 (Pin_4), J3.26
- net DSP-PWM7B: now also J10.7 (Pin_7), J3.36
- net DSP-PWM8A: now also J10.5 (Pin_5), J3.24
- net DSP-PWM8B: now also J10.8 (Pin_8), J3.43
- net DSP-PWM9A: now also J10.6 (Pin_6), J3.41
- net DSP-PWM9B: now also J10.9 (Pin_9), J3.22
- net DSP_A_CAN_EN: now also J9.44
- net DSP_A_CAN_RX: now also J9.37
- net DSP_A_CAN_TX: now also J9.39
- net DSP_B_CAN_EN: now also J9.17
- net DSP_B_CAN_RX: now also J9.24
- net DSP_B_CAN_TX: now also J9.15
- net DSP_Discharge1_EN: now also J4.44
- net DSP_Discharge2_EN: now also J4.42
- net DSP_PWM1_~{FAULT}: now also J4.35
- net DSP_PWM1~{_ENABL}E: now also R291.2
- net DSP_PWM2_~{FAULT}: now also J4.29
- net DSP_PWM2~{_ENABL}E: now also R292.2
- net DSP_Temperature1: now also J4.21
- net DSP_Temperature2: now also J4.31
- net DSP_VDC_BUS1: now also J18.3 (Pin_3)
- net DSP_VDC_BUS2: now also J18.4 (Pin_4)
- net GND: now also C136.2, DSUB3.8, DSUB3.9, J10.18 (Pin_18), J10.19 (Pin_19), J10.20 (Pin_20), J14.18 (Pin_18), J14.19 (Pin_19), J14.20 (Pin_20), J3.1, J3.17, J3.33, J3.49, J4.1, J4.17, J4.33, J4.49, J9.1, J9.25, J9.49, Q57.7 (GND)
- net GPIO100: now also J3.25
- net GPIO101: now also J3.14
- net GPIO102: now also J3.23
- net GPIO103: now also J3.21
- net GPIO104: now also J3.12
- net GPIO105: now also J3.15
- net GPIO107: now also J3.28, J3.3, Q57.1 (1A)
- net GPIO108: now also J3.44, J3.5, Q57.3 (2A)
- net GPIO109: now also J3.4, J3.45, Q57.5 (3A)
- net GPIO110: now also J3.6
- net GPIO115: now also J9.30
- net GPIO116: now also J9.46
- net GPIO117: now also J9.35
- net GPIO119: now also J9.19
- net GPIO127: now also J9.36
- net GPIO129: now also J9.41
- net GPIO137: now also J9.10
- net GPIO138: now also J9.14
- net GPIO147: now also J4.16
- net GPIO149: now also J4.39
- net GPIO157: now also J4.12
- net GPIO158: now also J4.37
- net GPIO24: now also J3.9
- net GPIO25: now also J3.10
- net GPIO26: now also SPI2.7 (Pin_7), J3.13; no longer SPI2.8 (Pin_8)
- net GPIO27: now also SPI2.8 (Pin_8), J3.7; no longer SPI2.7 (Pin_7)
- net GPIO28: now also J9.32
- net GPIO32: now also J9.31
- net GPIO33: now also J9.29
- net GPIO34: now also J9.27
- net GPIO35: now also J9.23
- net GPIO36: now also J9.20
- net GPIO42: now also J4.20
- net GPIO43: now also J4.47
- net GPIO48: now also J9.11
- net GPIO49: now also J9.5
- net GPIO50: now also J9.8
- net GPIO51: now also J9.12
- net GPIO53: now also J4.48
- net GPIO54: now also J9.6, Q57.13 (6A)
- net GPIO55: now also J9.3, Q57.11 (5A)
- net GPIO56: now also J4.40
- net GPIO57: now also J9.4, Q57.9 (4A)
- net GPIO58: now also J4.38
- net GPIO59: now also J4.28
- net GPIO60: now also J4.30
- net GPIO61: now also J4.26
- net GPIO67: now also J4.43
- net GPIO86: now also J4.41
- net GPIO89: now also J4.3
- net GPIO90: now also J4.9
- net GPIO91: now also J4.4
- net GPIO92: now also J4.5
- net GPIO93: now also J3.48
- net GPIO94: now also J3.42
- net GPIO99: now also J3.29
- net PE_GND: now also DSUB3.16, DSUB3.17
- net VDD: now also C136.1, J10.3 (Pin_3), J14.3 (Pin_3), Q57.14 (VCC), R291.1, R292.1
- net HALL_U renamed HALL1_U
- net HALL_UY renamed HALL1_UY
- net HALL_U_H renamed HALL1_U_H
- net HALL_U_L renamed HALL1_U_L
- net HALL_V renamed HALL1_V
- net HALL_VY renamed HALL1_VY
- net HALL_V_H renamed HALL1_V_H
- net HALL_V_L renamed HALL1_V_L
- net HALL_W renamed HALL1_W
- net HALL_WY renamed HALL1_WY
- net HALL_W_H renamed HALL1_W_H
- net HALL_W_L renamed HALL1_W_L
- net LED4 renamed GPIO118
- net GPIO118: now also J9.33
- new net 485_RTS_3: J4.13
- new net 485_RTS_4: J3.8
- new net ADC_DO_V_3: J10.12 (Pin_12), J16.3 (Pin_3)
- new net ADC_DO_V_4: J14.12 (Pin_12), J15.3 (Pin_3)
- new net ADC_DO_W_3: J10.13 (Pin_13), J9.48
- new net ADC_DO_W_4: J14.13 (Pin_13), J9.9
- new net DSP_Discharge3_EN: J10.15 (Pin_15), J4.36
- new net DSP_Discharge4_EN: J14.15 (Pin_15), J4.32
- new net DSP_PWM1~{_ENABLE}: J3.32
- new net DSP_PWM2~{_ENABLE}: J3.47
- new net DSP_PWM3_~{FAULT}: J10.17 (Pin_17), J4.14
- new net DSP_PWM3~{_ENABLE}: J10.10 (Pin_10), J3.40
- new net DSP_PWM4_~{FAULT}: J14.17 (Pin_17), J4.45
- new net DSP_PWM4~{_ENABLE}: J14.10 (Pin_10), J3.35
- new net DSP_Temperature3: J10.16 (Pin_16), J4.10
- new net DSP_Temperature4: J14.16 (Pin_16), J3.46
- new net DSP_VDC_BUS3: J10.14 (Pin_14), J17.3 (Pin_3)
- new net DSP_VDC_BUS4: J14.14 (Pin_14), J17.4 (Pin_4)
- new net GPIO125: J9.45
- new net GPIO126: J16.1 (Pin_1), J16.2 (Pin_2), J9.47
- new net GPIO134: J15.1 (Pin_1), J15.2 (Pin_2), J9.16
- new net HALL2_U: Q57.2 (1Y)
- new net HALL2_U_H: DSUB3.3
- new net HALL2_U_L: DSUB3.2
- new net HALL2_V: Q57.4 (2Y)
- new net HALL2_V_H: DSUB3.6
- new net HALL2_V_L: DSUB3.7
- new net HALL2_W: Q57.6 (3Y)
- new net HALL2_W_H: DSUB3.11
- new net HALL2_W_L: DSUB3.12
- new net MQEP2A: Q57.12 (6Y)
- new net MQEP2A_H: DSUB3.15
- new net MQEP2A_L: DSUB3.10
- new net MQEP2B: Q57.10 (5Y)
- new net MQEP2B_H: DSUB3.5
- new net MQEP2B_L: DSUB3.4
- new net MQEP2Z: Q57.8 (4Y)
- new net MQEP2Z_H: DSUB3.13
- new net MQEP2Z_L: DSUB3.14
- no-connect marks 14 -> 17
Other:
- added sheet H_485_3 (H485.kicad_sch)
- added sheet H_485_4 (H485.kicad_sch)
- added sheet 差分输入2 (26c32.kicad_sch)
- sheet H_485_1 ports: added 485A, 485B; removed none
- sheet H_485_2 ports: added 485A, 485B; removed none
- note added: "A"
- note added: "B"
- note added: "C"
- note added: "D"
- note removed: "BOOT"
- note removed: "DELETE"
- moved on the sheet: R287, R288

Commit message: 修改了一些bug，进行了一些布线
Parts:
- removed J3, J4, J9: ~, 1mmlab_footprint:CONN-SMD_50P-P0.50_XKB_X0515WVS-50AS-9TV01, symbol 1mmlab:X0515WVS-50AS-9TV01
- removed U1: ~, 1mmlab_footprint:CONN-SMD_50P-P0.50_XKB_X0515FVS-50CS-9TV01, symbol 1mmlab:X0515FVS-50AS-9TV01
- added J2, J3, J4, J5: ~, 1mmlab_footprint:CONN-SMD_50P-P0.50_XKB_X0515FVS-50CS-9TV01, symbol 1mmlab:X0515FVS-50AS-9TV01
- J1: renamed from J18; footprint (none) -> Connector_PinHeader_2.54mm:PinHeader_2x02_P2.54mm_Vertical_SMD
- J11: renamed from J10; footprint (none) -> Connector_PinHeader_2.54mm:PinHeader_2x10_P2.54mm_Vertical_SMD
- J12: renamed from J14; footprint (none) -> Connector_PinHeader_2.54mm:PinHeader_2x10_P2.54mm_Vertical_SMD
- J6: renamed from J17; footprint (none) -> Connector_PinHeader_2.54mm:PinHeader_2x02_P2.54mm_Vertical_SMD
- J7: renamed from J16; footprint (none) -> Connector_PinHeader_2.54mm:PinHeader_2x02_P2.54mm_Vertical_SMD
- J8: renamed from J15; footprint (none) -> Connector_PinHeader_2.54mm:PinHeader_2x02_P2.54mm_Vertical_SMD
- renumbered C215 to C1, C130 to C10, C131 to C11, C132 to C12, C133 to C13, C134 to C14, C135 to C15, C119 to C16, C120 to C17, C138 to C18, C140 to C19, C122 to C2, C121 to C20, C136 to C21, C142 to C22, C143 to C23, C144 to C24, C123 to C3, C124 to C4, C125 to C5, C126 to C6, C127 to C7, C128 to C8, C129 to C9, CN9 to CN1, CN10 to CN2, D31 to D1, D42 to D10, D43 to D11, D39 to D12, D44 to D13, D37 to D2, D38 to D3, D25 to D4, D28 to D5, D29 to D6, D26 to D7, D41 to D8, D27 to D9, DSUB3 to DSUB2, J7 to J10, J1 to J13, J8 to J14, J5 to J15, J11 to J16, J6 to J9, L17 to L1, L18 to L2, Q48 to Q1, Q49 to Q2, Q50 to Q3, Q51 to Q4, Q56 to Q5, Q57 to Q6, Q52 to Q7, Q47 to Q8, Q53 to Q9, R366 to R1, R308 to R10, R309 to R11, R310 to R12, R311 to R13, R291 to R14, R292 to R15, R287 to R16, R288 to R17, R312 to R18, R313 to R19, R300 to R2, R314 to R20, R268 to R21, R269 to R22, R315 to R23, R270 to R24, R271 to R25, R316 to R26, R317 to R27, R318 to R28, R319 to R29, R301 to R3, R320 to R30, R321 to R31, R322 to R32, R323 to R33, R302 to R4, R303 to R5, R304 to R6, R305 to R7, R306 to R8, R307 to R9, SPI2 to SPI1, SPI3 to SPI2, SPI4 to SPI3
Connections:
- net DSP_PWM1~{_ENABL}E is gone; now on net DSP_PWM1~{_ENABLE}: R14.2
- net DSP_PWM2~{_ENABL}E is gone; now on net DSP_PWM2~{_ENABLE}: R15.2
- net DSP_PWM3~{_ENABL}E is gone; now on net DSP_PWM3~{_ENABLE}: R16.2
- net DSP_PWM4~{_ENABL}E is gone; now on net DSP_PWM4~{_ENABLE}: R17.2
- net HALL1_U is gone; now on net GPIO107: Q5.2 (1Y)
- net HALL1_V is gone; now on net GPIO108: Q5.4 (2Y)
- net HALL1_W is gone; now on net GPIO109: Q5.6 (3Y)
- net MQEP1A is gone; now on net GPIO50: Q5.12 (6Y)
- net MQEP1B is gone; now on net GPIO51: Q5.10 (5Y)
- net MQEP1Z is gone; now on net GPIO53: Q5.8 (4Y)
- net MQEP2A is gone; now on net GPIO54: Q6.12 (6Y)
- net MQEP2B is gone; now on net GPIO55: Q6.10 (5Y)
- net MQEP2Z is gone; now on net GPIO57: Q6.8 (4Y)
- net 485_RTS_1: now also J5.43
- net 485_RTS_2: now also J4.28
- net 485_RTS_3: now also J4.37
- net 485_RTS_4: now also J3.44
- net ADC_14_IN: now also J2.23
- net ADC_15_IN: now also J2.19
- net ADC_A0_IN: now also J2.47
- net ADC_A1_IN: now also J2.43
- net ADC_A2_IN: now also J2.39
- net ADC_A3_IN: now also J2.35
- net ADC_A4_IN: now also J2.31
- net ADC_A5_IN: now also J2.27
- net ADC_B0_IN: now also J2.48
- net ADC_B1_IN: now also J2.44
- net ADC_B2_IN: now also J2.40
- net ADC_B3_IN: now also J2.36
- net ADC_B4_IN: now also J2.32
- net ADC_B5_IN: now also J2.28
- net ADC_C2_IN: now also J2.15
- net ADC_C3_IN: now also J2.11
- net ADC_C4_IN: now also J2.7
- net ADC_C5_IN: now also J2.3
- net ADC_CLK_X1: now also J5.10
- net ADC_CLK_X2: now also J5.18
- net ADC_D0_IN: now also J2.24
- net ADC_D1_IN: now also J2.20
- net ADC_D2_IN: now also J2.16
- net ADC_D3_IN: now also J2.12
- net ADC_D4_IN: now also J2.8
- net ADC_D5_IN: now also J2.4
- net ADC_DO_V_1: now also J5.12
- net ADC_DO_V_2: now also J5.7
- net ADC_DO_W_1: now also J5.14
- net ADC_DO_W_2: now also J5.30
- net ADC_DO_W_3: now also J5.4
- net ADC_DO_W_4: now also J5.41
- net CAN_H1: now also D3.2; no longer D3.1
- net CAN_H2: now also D2.2; no longer D2.1
- net CAN_L1: now also D3.1; no longer D3.2
- net CAN_L2: now also D2.1; no longer D2.2
- net D+5V: now also J3.18, J3.2, J3.34, J3.50, J4.18, J4.2, J4.34, J4.50, J5.2, J5.26, J5.50
- net DI-1-DSP-3.3V: now also J5.29, J5.34
- net DI-2-DSP-3.3V: now also J5.24, J5.37
- net DSP-PWM10A: now also J3.13
- net DSP-PWM10B: now also J3.11
- net DSP-PWM11A: now also J3.32
- net DSP-PWM11B: now also J3.19
- net DSP-PWM12A: now also J3.31
- net DSP-PWM12B: now also J3.39
- net DSP-PWM1A: now also J4.23
- net DSP-PWM1B: now also J4.35
- net DSP-PWM2A: now also J4.39
- net DSP-PWM2B: now also J4.44
- net DSP-PWM3A: now also J4.31
- net DSP-PWM3B: now also J4.43
- net DSP-PWM4A: now also J4.27
- net DSP-PWM4B: now also J4.46
- net DSP-PWM5A: now also J3.36
- net DSP-PWM5B: now also J3.23
- net DSP-PWM6A: now also J3.22
- net DSP-PWM6B: now also J3.14
- net DSP-PWM7A: now also J3.26
- net DSP-PWM7B: now also J3.16
- net DSP-PWM8A: now also J3.28
- net DSP-PWM8B: now also J3.7
- net DSP-PWM9A: now also J3.9
- net DSP-PWM9B: now also J3.30
- net DSP_A_CAN_EN: now also J5.8
- net DSP_A_CAN_RX: now also J5.13
- net DSP_A_CAN_TX: now also J5.11
- net DSP_B_CAN_EN: now also J5.33
- net DSP_B_CAN_RX: now also J5.28
- net DSP_B_CAN_TX: now also J5.35
- net DSP_Discharge1_EN: now also J4.8
- net DSP_Discharge2_EN: now also J4.10
- net DSP_Discharge3_EN: now also J4.16
- net DSP_Discharge4_EN: now also J4.20
- net DSP_PWM1_~{FAULT}: now also J4.15
- net DSP_PWM1~{_ENABLE}: now also J3.20
- net DSP_PWM2_~{FAULT}: now also J4.21
- net DSP_PWM2~{_ENABLE}: now also J3.3
- net DSP_PWM3_~{FAULT}: now also J4.38
- net DSP_PWM3~{_ENABLE}: now also J3.12
- net DSP_PWM4_~{FAULT}: now also J4.5
- net DSP_PWM4~{_ENABLE}: now also J3.15
- net DSP_Temperature1: now also J4.29
- net DSP_Temperature2: now also J4.19
- net DSP_Temperature3: now also J4.42
- net DSP_Temperature4: now also J3.6
- net GND: now also C7.2, Q8.1 (GND), J2.1, J2.10, J2.13, J2.14, J2.17, J2.18, J2.2, J2.21, J2.22, J2.25, J2.26, J2.29, J2.30, J2.33, J2.34, J2.37, J2.38, J2.41, J2.42, J2.45, J2.46, J2.49, J2.5, J2.50, J2.6, J2.9, J3.1, J3.17, J3.33, J3.49, J4.1, J4.17, J4.33, J4.49, J5.1, J5.25, J5.49
- net GPIO100: now also J3.25
- net GPIO101: now also J3.38
- net GPIO102: now also J3.27
- net GPIO103: now also J3.29
- net GPIO104: now also J3.40
- net GPIO105: now also J3.35
- net GPIO107: now also J3.47; no longer Q6.1 (1A)
- net GPIO108: now also J3.45; no longer Q6.3 (2A)
- net GPIO109: now also J3.48; no longer Q6.5 (3A)
- net GPIO110: now also J3.46
- net GPIO115: now also J5.22
- net GPIO116: now also J5.6
- net GPIO117: now also J5.15
- net GPIO118: now also J5.17
- net GPIO119: now also J5.31
- net GPIO125: now also J5.5
- net GPIO126: now also J5.3
- net GPIO127: now also J5.16
- net GPIO129: now also J5.9
- net GPIO134: now also J5.36
- net GPIO137: now also J5.42
- net GPIO138: now also J5.38
- net GPIO147: now also J4.36
- net GPIO149: now also J4.11
- net GPIO157: now also J4.40
- net GPIO158: now also J4.13
- net GPIO24: now also J3.41
- net GPIO25: now also J3.42
- net GPIO26: now also J3.37
- net GPIO27: now also J3.43
- net GPIO28: now also J5.20
- net GPIO32: now also J5.19
- net GPIO33: now also J5.21
- net GPIO34: now also J5.23
- net GPIO35: now also J5.27
- net GPIO36: now also J5.32
- net GPIO42: now also J4.32
- net GPIO43: now also J4.3
- net GPIO48: now also J5.39
- net GPIO49: now also J5.45
- net GPIO50: now also J5.44; no longer Q5.13 (6A)
- net GPIO51: now also J5.40; no longer Q5.11 (5A)
- net GPIO53: now also J4.4; no longer Q5.9 (4A)
- net GPIO54: now also J5.46; no longer Q6.13 (6A)
- net GPIO55: now also J5.47; no longer Q6.11 (5A)
- net GPIO56: now also J4.12
- net GPIO57: now also J5.48; no longer Q6.9 (4A)
- net GPIO58: now also J4.14
- net GPIO59: now also J4.24
- net GPIO60: now also J4.22
- net GPIO61: now also J4.26
- net GPIO67: now also J4.7
- net GPIO86: now also J4.9
- net GPIO89: now also J4.47
- net GPIO90: now also J4.41
- net GPIO91: now also J4.48
- net GPIO92: now also J4.45
- net GPIO93: now also J3.4
- net GPIO94: now also J3.10
- net GPIO99: now also J3.21
- net HALL2_U renamed GPIO166
- net GPIO166: now also J3.24
- net HALL2_V renamed GPIO167
- net GPIO167: now also J3.8
- net HALL2_W renamed GPIO168
- net GPIO168: now also J3.5
- new net HALL2_UY: Q6.1 (1A)
- new net HALL2_VY: Q6.3 (2A)
- new net HALL2_WY: Q6.5 (3A)
- new net MQEP1AY: Q5.13 (6A)
- new net MQEP1BY: Q5.11 (5A)
- new net MQEP1ZY: Q5.9 (4A)
- new net MQEP2AY: Q6.13 (6A)
- new net MQEP2BY: Q6.11 (5A)
- new net MQEP2ZY: Q6.9 (4A)
- no-connect marks 17 -> 26
Other:
- removed sheet 差分输入
- added sheet 差分输入3 (26c32.kicad_sch)
- added sheet 差分输入4 (26c32.kicad_sch)
- moved on the sheet: C10, C11, C12, C13, C2, C3, C4, C5, C6, C7, C8, C9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

Commit message: 基本完成初步的布线，但是额外逆变器接口位置极不合理，需要返工
Parts:
- removed J7, J8: Conn_02x02_Top_Bottom, Connector_PinHeader_2.54mm:PinHeader_2x02_P2.54mm_Vertical_SMD, symbol Connector_Generic:Conn_02x02_Top_Bottom
- added R184, R186: 0R, Lib_sheet_10:R_0603_1608Metric, symbol sheet1-altium-import:RES_2
- added R185, R187: DNP, Lib_sheet_10:R_0603_1608Metric, symbol sheet1-altium-import:RES_2
- J1, J6: footprint Connector_PinHeader_2.54mm:PinHeader_2x02_P2.54mm_Vertical_SMD -> Connector_PinHeader_1.27mm:PinHeader_2x02_P1.27mm_Vertical_SMD
- J11, J12: footprint Connector_PinHeader_2.54mm:PinHeader_2x10_P2.54mm_Vertical_SMD -> Connector_PinHeader_1.27mm:PinHeader_2x10_P1.27mm_Vertical_SMD
Connections:
- net GPIO110 is gone; now on net DSP_Temperature2: J3.46
- net GPIO125 is gone; now on net DSP_PWM3_~{FAULT}: J5.5
- net GPIO127 is gone; now on net DSP_Discharge3_EN: J5.16
- net GPIO56 is gone; now on net DSP_Temperature1: J4.12
- net ADC_DO_U_1: now also R186.1
- net ADC_DO_U_2: now also R185.2
- net ADC_DO_V_3: now also R187.1
- net ADC_DO_V_4: now also R184.2
- net DI-1-DSP-3.3V: no longer J5.34
- net DI-2-DSP-3.3V: no longer J5.24
- net DSP_Discharge2_EN: now also J3.47; no longer J4.10
- net DSP_Discharge3_EN: no longer J4.16
- net DSP_PWM1~{_ENABLE}: now also J5.34; no longer J3.20
- net DSP_PWM2_~{FAULT}: now also J3.48; no longer J4.21
- net DSP_PWM2~{_ENABLE}: now also J3.45; no longer J3.3
- net DSP_PWM3_~{FAULT}: no longer J4.38
- net DSP_PWM3~{_ENABLE}: now also J3.20; no longer J3.12
- net DSP_Temperature1: no longer J4.29
- net DSP_Temperature2: no longer J4.19
- net GPIO126: now also R186.2, R187.2
- net GPIO134: now also R184.1, R185.1
- net GPIO147: now also Q6.4 (2Y)
- net GPIO157: now also Q6.2 (1Y)
- net GPIO166: now also Q5.6 (3Y); no longer Q6.2 (1Y)
- net GPIO167: now also Q5.4 (2Y); no longer Q6.4 (2Y)
- net GPIO168: now also Q5.2 (1Y); no longer Q6.6 (3Y)
- net GPIO42: now also Q6.6 (3Y)
- net GPIO50: no longer Q5.12 (6Y)
- net GPIO51: no longer Q5.10 (5Y)
- net GPIO53: no longer Q5.8 (4Y)
- net GPIO99: now also Q5.8 (4Y)
- removed net GPIO107: J3.47, Q5.2 (1Y)
- removed net GPIO108: J3.45, Q5.4 (2Y)
- removed net GPIO109: J3.48, Q5.6 (3Y)
- new net GPIO121: J5.24
- new net GPIO140: J4.10
- new net GPIO141: J4.16
- new net GPIO153: J4.21
- new net GPIO154: J4.38
- new net GPIO162: J4.29
- new net GPIO163: J4.19
- new net GPIO96: J3.3, Q5.12 (6Y)
- new net GPIO97: J3.12, Q5.10 (5Y)
- no-connect marks 26 -> 25

Commit message: 完成布局布线，需要丝印检查，原理图检查
Parts:
- removed D4, D7: LEDRED, LED_SMD:LED_0805_2012Metric, symbol sheet1-altium-import:root_3_LED0
- removed Q3, Q4: FMMT618TA, Package_TO_SOT_SMD:SOT-23, symbol sheet1-altium-import:root_0_NPN
- removed R18, R23: 10K, Resistor_SMD:R_0805_2012Metric, symbol sheet1-altium-import:root_2_Res2
- removed R19, R26: 2K, Resistor_SMD:R_0805_2012Metric, symbol sheet1-altium-import:root_3_Res2
- removed R20, R27: 1K, Resistor_SMD:R_0805_2012Metric, symbol sheet1-altium-import:root_1_Res2
- added J18: Conn_02x12_Odd_Even, 1mmlab_footprint:CONN-TH_24P-P2.00_XUNPU_PHB2.0-02-24PZZ, symbol Connector_Generic:Conn_02x12_Odd_Even
Connections:
- net GPIO117 is gone; now on net DSP_PWM4_~{FAULT}: J5.15
- net GPIO118 is gone; now on net DSP_Discharge4_EN: J5.17
- net GPIO121 is gone; now on net DSP_Temperature4: J5.24
- net GPIO129 is gone; now on net DSP_Temperature3: J5.9
- net GPIO28 is gone; now on net DSP_PWM4~{_ENABLE}: J5.20
- net ADC_14_IN: now also J18.14 (Pin_14)
- net ADC_15_IN: now also J18.16 (Pin_16)
- net ADC_A0_IN: now also J18.2 (Pin_2)
- net ADC_A1_IN: now also J18.4 (Pin_4)
- net ADC_A2_IN: now also J18.6 (Pin_6)
- net ADC_A3_IN: now also J6.2 (Pin_2), J18.8 (Pin_8); no longer J6.1 (Pin_1)
- net ADC_A4_IN: now also J6.1 (Pin_1), J18.10 (Pin_10); no longer J6.2 (Pin_2)
- net ADC_A5_IN: now also J18.12 (Pin_12)
- net ADC_B0_IN: now also J18.1 (Pin_1)
- net ADC_B1_IN: now also J18.3 (Pin_3)
- net ADC_B2_IN: now also J18.5 (Pin_5)
- net ADC_B3_IN: now also J18.7 (Pin_7)
- net ADC_B4_IN: now also J18.9 (Pin_9)
- net ADC_B5_IN: now also J18.11 (Pin_11)
- net ADC_C2_IN: now also J18.18 (Pin_18)
- net ADC_C3_IN: now also J18.20 (Pin_20)
- net ADC_C4_IN: now also J18.22 (Pin_22)
- net ADC_C5_IN: now also J18.24 (Pin_24)
- net ADC_D0_IN: now also J18.13 (Pin_13)
- net ADC_D1_IN: now also J18.15 (Pin_15)
- net ADC_D2_IN: now also J18.17 (Pin_17)
- net ADC_D3_IN: now also J18.19 (Pin_19)
- net ADC_D4_IN: now also J18.21 (Pin_21)
- net ADC_D5_IN: now also J18.23 (Pin_23)
- net DSP_Discharge4_EN: no longer J4.20
- net DSP_PWM4_~{FAULT}: no longer J4.5
- net DSP_PWM4~{_ENABLE}: no longer J3.15
- net DSP_Temperature3: no longer J4.42
- net DSP_Temperature4: no longer J3.6
- net DSP_VDC_BUS3: now also J6.4 (Pin_4); no longer J6.3 (Pin_3)
- net DSP_VDC_BUS4: now also J6.3 (Pin_3); no longer J6.4 (Pin_4)
- new net GPIO142: J4.20
- new net GPIO155: J4.5
- new net GPIO164: J4.42
- new net GPIO165: J3.6
- new net GPIO98: J3.15
