File: 28388motherboard/26c32.kicad_sch (KiCad schematic)
At the start: 38 parts, among them Q47 AM26C32CD

Commit message: 底板分配引脚
Parts:
- removed D65, D66, D71, D72, D77, D78: ${MANUFACTURER PART}, 1mmlab_footprint:SOD-323_L1.8-W1.3-LS2.5-BI, symbol ESD:PESD12VL1BA,115
- added D14, D16, D18: SDT23C712L02_C5197393, Lib2ic:SOT-23-3_L2.9-W1.3-P1.90-LS2.4-BR, symbol sheet1-altium-import:SDT23C712L02_C5197393
- renumbered C184 to C205, C185 to C206, C186 to C208, C187 to C211, C188 to C213, C189 to C214, C190 to C218, C191 to C219, C192 to C221, C193 to C223, L16 to L22, L17 to L24, L18 to L26, Q47 to Q54, R291 to R327, R292 to R330, R293 to R331, R294 to R334, R295 to R336, R296 to R337, R297 to R340, R298 to R341, R299 to R343, R300 to R346, R301 to R347, R302 to R350, R303 to R351, R304 to R353, R305 to R355, R306 to R358, R307 to R359, R308 to R362
Connections:
- net GND: now also D14.3, D16.3, D18.3
- net at C214.1, C221.1, L26.2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: now also D18.2
- net at C208.1, C214.2, L26.3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: now also D18.1
- net at C213.1, C219.1, L24.3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: now also D16.2
- net at C205.1, C211.2, L22.3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: now also D14.2
- net at C206.1, C213.2, L24.2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: now also D16.1
- net at C211.1, C218.1, L22.2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: now also D14.1

Commit message: 修改了一些bug，进行了一些布线
Parts:
- renumbered C205 to C45, C206 to C46, C208 to C47, C211 to C48, C213 to C49, C214 to C50, C218 to C51, C219 to C52, C221 to C53, C223 to C54, D14 to D20, D16 to D21, D18 to D22, L22 to L5, L24 to L6, L26 to L7, Q54 to Q20, R351 to R100, R353 to R101, R355 to R102, R358 to R103, R359 to R104, R362 to R105, R327 to R88, R330 to R89, R331 to R90, R334 to R91, R336 to R92, R337 to R93, R340 to R94, R341 to R95, R343 to R96, R346 to R97, R347 to R98, R350 to R99
Connections:
- no-connect marks 3 -> 10

Commit message: 基本完成初步的布线，但是额外逆变器接口位置极不合理，需要返工
Connections:
- net at C50.1, C53.1, L7.2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: now also D22.1; no longer D22.2
- net at C47.1, C50.2, L7.3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: now also D22.2; no longer D22.1
- no-connect marks 10 -> 7
Changed lines of the file:
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@@
-	)
-	(junction
-		(at 105.41 124.46)
-		(diameter 0)
-		(color 0 0 0 0)
 	)
 	(junction
@@
 	)
 	(junction
-		(at 99.06 130.81)
-		(diameter 0)
-		(color 0 0 0 0)
-	)
-	(junction
 		(at 118.11 63.5)
 		(diameter 0)
@@
 	)
 	(junction
+		(at 105.41 130.81)
+		(diameter 0)
+		(color 0 0 0 0)
+	)
+	(junction
 		(at 118.11 50.8)
 		(diameter 0)
@@
 	(junction
 		(at 99.06 96.52)
+		(diameter 0)
+		(color 0 0 0 0)
+	)
+	(junction
+		(at 99.06 124.46)
 		(diameter 0)
 		(color 0 0 0 0)
@@
 	)
 	(no_connect
-		(at 127 36.83)
-	)
-	(no_connect
-		(at 130.81 38.1)
-	)
-	(no_connect
-		(at 142.24 43.18)
-	)
-	(no_connect
 		(at 214.63 62.23)
 	)
@@
 	(wire
 		(pts
+			(xy 99.06 124.46) (xy 99.06 140.97)
+		)
+		(stroke
+			(width 0)
+			(type default)
+		)
+	)
+	(wire
+		(pts
 			(xy 167.64 82.55) (xy 175.26 82.55)
 		)
@@
 	(wire
 		(pts
-			(xy 99.06 130.81) (xy 114.3 130.81)
+			(xy 97.79 130.81) (xy 105.41 130.81)
 		)
 		(stroke
@@
 	(wire
 		(pts
-			(xy 105.41 124.46) (xy 109.22 124.46)
-		)
-		(stroke
-			(width 0)
-			(type default)
-		)
-	)
-	(wire
-		(pts
 			(xy 205.74 46.99) (xy 205.74 52.07)
 		)
@@
 	(wire
 		(pts
-			(xy 99.06 140.97) (xy 99.06 130.81)
-		)
-		(stroke
-			(width 0)
-			(type default)
-		)
-	)
-	(wire
-		(pts
 			(xy 118.11 118.11) (xy 121.92 118.11)
 		)
@@
 	(wire
 		(pts
-			(xy 97.79 130.81) (xy 99.06 130.81)
-		)
-		(stroke
-			(width 0)
-			(type default)
-		)
-	)
-	(wire
-		(pts
 			(xy 114.3 146.05) (xy 121.92 146.05)
 		)
@@
 	(wire
 		(pts
+			(xy 105.41 130.81) (xy 114.3 130.81)
+		)
+		(stroke
+			(width 0)
+			(type default)
+		)
+	)
+	(wire
+		(pts
 			(xy 121.92 63.5) (xy 121.92 66.04)
 		)
@@
 	(wire
 		(pts
+			(xy 99.06 124.46) (xy 109.22 124.46)
+		)
+		(stroke
+			(width 0)
+			(type default)
+		)
+	)
+	(wire
+		(pts
 			(xy 114.3 111.76) (xy 121.92 111.76)
 		)
@@
 	(wire
 		(pts
-			(xy 105.41 146.05) (xy 105.41 124.46)
-		)
-		(stroke
-			(width 0)
-			(type default)
-		)
-	)
-	(wire
-		(pts
 			(xy 121.92 83.82) (xy 125.73 83.82)
 		)
@@
 	(wire
 		(pts
-			(xy 97.79 124.46) (xy 105.41 124.46)
+			(xy 97.79 124.46) (xy 99.06 124.46)
 		)
 		(stroke
@@
 		)
 		(stroke
+			(width 0)
+			(type default)
+		)
+	)
+	(wire
+		(pts
+			(xy 105.41 130.81) (xy 105.41 146.05)
+		)
+		(stroke
